File: motorgo_plink/LISM6.kicad_sch (KiCad schematic)
At the start: 20 parts, among them J23 Conn_01x06_Pin, U10 LIS3MDLTR, U11 LSM6DS3TR

Commit message: WIP - adding P/Ns to BOM (TS). will finish in afternoon.
Parts:
- C30, C31: footprint Capacitor_SMD:C_01005_0402Metric -> Capacitor_SMD:C_0402_1005Metric; Field4 (none) -> updated footprint TS 05-31. if 50V needed, see C3; LCSC_Part_Number (none) -> C880603
- C32: LCSC_Part_Number (none) -> C15849
Changed lines of the file:
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@@
       (effects (font (size 1.27 1.27)))
     )
-    (property "Footprint" "Capacitor_SMD:C_01005_0402Metric" (at 59.055 118.745 0)
-      (effects (font (size 1.27 1.27)) hide)
-    )
-    (property "Datasheet" "~" (at 59.055 118.745 0)
+    (property "Footprint" "Capacitor_SMD:C_0402_1005Metric" (at 59.055 118.745 0)
+      (effects (font (size 1.27 1.27)) hide)
+    )
+    (property "Datasheet" "https://www.lcsc.com/product-detail/Multilayer-Ceramic-Capacitors-MLCC-SMD-SMT_CCTC-TCC0402X5R104K250AT_C880603.html" (at 59.055 118.745 0)
+      (effects (font (size 1.27 1.27)) hide)
+    )
+    (property "Field4" "updated footprint TS 05-31. if 50V needed, see C3" (at 59.055 118.745 0)
+      (effects (font (size 1.27 1.27)) hide)
+    )
+    (property "LCSC_Part_Number" "C880603" (at 59.055 118.745 0)
       (effects (font (size 1.27 1.27)) hide)
     )
@@
       (effects (font (size 1.27 1.27)))
     )
-    (property "Footprint" "Capacitor_SMD:C_01005_0402Metric" (at 76.835 119.38 0)
-      (effects (font (size 1.27 1.27)) hide)
-    )
-    (property "Datasheet" "~" (at 76.835 119.38 0)
+    (property "Footprint" "Capacitor_SMD:C_0402_1005Metric" (at 76.835 119.38 0)
+      (effects (font (size 1.27 1.27)) hide)
+    )
+    (property "Datasheet" "https://www.lcsc.com/product-detail/Multilayer-Ceramic-Capacitors-MLCC-SMD-SMT_CCTC-TCC0402X5R104K250AT_C880603.html" (at 76.835 119.38 0)
+      (effects (font (size 1.27 1.27)) hide)
+    )
+    (property "Field4" "updated footprint TS 05-31. if 50V needed, see C3" (at 76.835 119.38 0)
+      (effects (font (size 1.27 1.27)) hide)
+    )
+    (property "LCSC_Part_Number" "C880603" (at 76.835 119.38 0)
       (effects (font (size 1.27 1.27)) hide)
     )
@@
       (effects (font (size 1.27 1.27)) hide)
     )
-    (property "Datasheet" "~" (at 82.55 119.38 0)
-      (effects (font (size 1.27 1.27)) hide)
-    )
+    (property "Datasheet" "https://www.lcsc.com/product-detail/Multilayer-Ceramic-Capacitors-MLCC-SMD-SMT_Samsung-Electro-Mechanics-CL10A105KB8NNNC_C15849.html" (at 82.55 119.38 0)
+      (effects (font (size 1.27 1.27)) hide)
+    )
+    (property "LCSC_Part_Number" "C15849" (at 82.55 119.38 0)
+      (effects (font (size 1.27 1.27)) hide)
+    )

Commit message: finished first pass on BOM. check 100uF cap and a couple others. TS
Parts:
- R34: footprint (none) -> Resistor_SMD:R_0402_1005Metric; LCSC_Part_Number (none) -> C2906858
- R38, R39: LCSC_Part_Number (none) -> C4109
- R46, R49, R50: LCSC_Part_Number (none) -> C2906899
- U10: LCSC_Part_Number (none) -> C478483
- U11: LCSC_Part_Number (none) -> C95230
Changed lines of the file:
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@@
       (effects (font (size 1.27 1.27)) hide)
     )
-    (property "Datasheet" "~" (at 71.12 57.785 0)
+    (property "Datasheet" "https://www.lcsc.com/product-detail/Chip-Resistor-Surface-Mount_UNI-ROYAL-Uniroyal-Elec-0402WGF2001TCE_C4109.html" (at 71.12 57.785 0)
+      (effects (font (size 1.27 1.27)) hide)
+    )
+    (property "LCSC_Part_Number" "C4109" (at 71.12 57.785 0)
       (effects (font (size 1.27 1.27)) hide)
     )
@@
       (effects (font (size 1.27 1.27)) hide)
     )
-    (property "Datasheet" "~" (at 175.26 123.825 0)
+    (property "Datasheet" "https://www.lcsc.com/product-detail/Chip-Resistor-Surface-Mount_FOJAN-FRC0402J102-TS_C2906899.html" (at 175.26 123.825 0)
+      (effects (font (size 1.27 1.27)) hide)
+    )
+    (property "LCSC_Part_Number" "C2906899" (at 175.26 123.825 0)
       (effects (font (size 1.27 1.27)) hide)
     )
@@
       (effects (font (size 1.27 1.27)) hide)
     )
-    (property "Datasheet" "~" (at 146.685 123.825 0)
+    (property "Datasheet" "https://www.lcsc.com/product-detail/Chip-Resistor-Surface-Mount_FOJAN-FRC0402J102-TS_C2906899.html" (at 146.685 123.825 0)
+      (effects (font (size 1.27 1.27)) hide)
+    )
+    (property "LCSC_Part_Number" "C2906899" (at 146.685 123.825 0)
       (effects (font (size 1.27 1.27)) hide)
     )
@@
       (effects (font (size 1.27 1.27)))
     )
-    (property "Footprint" "" (at 238.125 70.485 0)
-      (effects (font (size 1.27 1.27)) hide)
-    )
-    (property "Datasheet" "~" (at 238.125 70.485 0)
+    (property "Footprint" "Resistor_SMD:R_0402_1005Metric" (at 238.125 70.485 0)
+      (effects (font (size 1.27 1.27)) hide)
+    )
+    (property "Datasheet" "https://www.lcsc.com/product-detail/Chip-Resistor-Surface-Mount_FOJAN-FRC0402F0000TS_C2906858.html" (at 238.125 70.485 0)
+      (effects (font (size 1.27 1.27)) hide)
+    )
+    (property "LCSC_Part_Number" "C2906858" (at 238.125 70.485 0)
       (effects (font (size 1.27 1.27)) hide)
     )
@@
       (effects (font (size 1.27 1.27)) hide)
     )
-    (property "Datasheet" "http://www.szlcsc.com/product/details_485763.html" (at 110.49 85.0138 0)
+    (property "Datasheet" "https://www.lcsc.com/product-detail/Linear-Hall-Sensors_STMicroelectronics-LIS3MDLTR_C478483.html" (at 110.49 85.0138 0)
       (effects (font (size 1.27 1.27)) hide)
     )
@@
     )
     (property "uuid" "std:3c4a1927816047c0b32d8307cf40d91b" (at 110.49 88.1888 0)
+      (effects (font (size 1.27 1.27)) hide)
+    )
+    (property "LCSC_Part_Number" "C478483" (at 111.125 104.14 0)
       (effects (font (size 1.27 1.27)) hide)
     )
@@
       (effects (font (size 1.27 1.27)) hide)
     )
-    (property "Datasheet" "~" (at 76.2 57.785 0)
+    (property "Datasheet" "https://www.lcsc.com/product-detail/Chip-Resistor-Surface-Mount_UNI-ROYAL-Uniroyal-Elec-0402WGF2001TCE_C4109.html" (at 76.2 57.785 0)
+      (effects (font (size 1.27 1.27)) hide)
+    )
+    (property "LCSC_Part_Number" "C4109" (at 76.2 57.785 0)
       (effects (font (size 1.27 1.27)) hide)
     )
@@
       (effects (font (size 1.27 1.27)) hide)
     )
-    (property "Datasheet" "~" (at 227.965 92.075 0)
+    (property "Datasheet" "https://www.lcsc.com/product-detail/Chip-Resistor-Surface-Mount_FOJAN-FRC0402J102-TS_C2906899.html" (at 227.965 92.075 0)
+      (effects (font (size 1.27 1.27)) hide)
+    )
+    (property "LCSC_Part_Number" "C2906899" (at 227.965 92.075 0)
       (effects (font (size 1.27 1.27)) hide)
     )
@@
       (effects (font (size 1.27 1.27)) hide)
     )
-    (property "Datasheet" "http://www.szlcsc.com/product/details_96431.html" (at 211.455 103.5558 0)
+    (property "Datasheet" "https://www.lcsc.com/product-detail/Attitude-Sensor-Gyroscope_STMicroelectronics-LSM6DS3TR_C95230.html" (at 211.455 103.5558 0)
       (effects (font (size 1.27 1.27)) hide)
     )
@@
       (effects (font (size 1.27 1.27)) hide)
     )
+    (property "LCSC_Part_Number" "C95230" (at 211.455 109.22 0)
+      (effects (font (size 1.27 1.27)) hide)
+    )
