File: motorgo_plink/LISM6.kicad_sch (KiCad schematic)
At the start: 2 parts, among them U10 LSM6DS3TR, U6 LIS3MDLTR

Commit message: WIP update for BOM co-work
Parts:
- added J23: Conn_01x09_Pin, symbol Connector:Conn_01x09_Pin
Connections:
- net +3V3: now reaches U10.5 (VDDIO)
- net +3V3: now also U10.8 (VDD)
Changed lines of the file:
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@@
 (kicad_sch (version 20230121) (generator eeschema)
   (paper "A4")
+  (wire (pts (xy 170.18 78.105) (xy 170.18 81.28))
+    (stroke (width 0) (type default))
+  )
+  (wire (pts (xy 171.45 82.55) (xy 176.53 82.55))
+    (stroke (width 0) (type default))
+  )
+  (wire (pts (xy 176.53 82.55) (xy 177.165 81.915))
+    (stroke (width 0) (type default))
+  )
+  (wire (pts (xy 168.275 76.2) (xy 170.18 78.105))
+    (stroke (width 0) (type default))
+  )
+  (wire (pts (xy 147.955 91.44) (xy 143.51 91.44))
+    (stroke (width 0) (type default))
+  )
+  (wire (pts (xy 167.64 76.2) (xy 168.275 76.2))
+    (stroke (width 0) (type default))
+  )
+  (wire (pts (xy 170.18 81.28) (xy 171.45 82.55))
+    (stroke (width 0) (type default))
+  )
+  (wire (pts (xy 148.59 85.09) (xy 148.59 90.805))
+    (stroke (width 0) (type default))
+  )
+  (wire (pts (xy 141.605 88.265) (xy 141.605 89.535))
+    (stroke (width 0) (type default))
+  )
+  (wire (pts (xy 148.59 90.805) (xy 147.955 91.44))
+    (stroke (width 0) (type default))
+  )
+  (wire (pts (xy 143.51 91.44) (xy 141.605 89.535))
+    (stroke (width 0) (type default))
+  )
+  (symbol (lib_id "power:GND") (at 151.765 92.71 0) (unit 1)
+    (in_bom yes) (on_board yes) (dnp no) (fields_autoplaced)
+    (property "Reference" "#PWR090" (at 151.765 99.06 0)
+      (effects (font (size 1.27 1.27)) hide)
+    )
+    (property "Value" "GND" (at 151.765 97.79 0)
+      (effects (font (size 1.27 1.27)))
+    )
+    (property "Footprint" "" (at 151.765 92.71 0)
+      (effects (font (size 1.27 1.27)) hide)
+    )
+    (property "Datasheet" "" (at 151.765 92.71 0)
+      (effects (font (size 1.27 1.27)) hide)
+    )
+    (pin "1")
+    (instances
+      (project "motorgo_plink"
+        (path "/e63e39d7-6ac0-4ffd-8aa3-1841a4541b55/7d6efa12-7b94-467b-977c-f0e88b0f6fad"
+          (reference "#PWR090") (unit 1)
+        )
+      )
+    )
+  )
+  (symbol (lib_id "Connector:Conn_01x09_Pin") (at 205.74 73.025 0) (unit 1)
+    (in_bom yes) (on_board yes) (dnp no) (fields_autoplaced)
+    (property "Reference" "J23" (at 206.375 57.15 0)
+      (effects (font (size 1.27 1.27)))
+    )
+    (property "Value" "Conn_01x09_Pin" (at 206.375 59.69 0)
+      (effects (font (size 1.27 1.27)))
+    )
+    (property "Footprint" "" (at 205.74 73.025 0)
+      (effects (font (size 1.27 1.27)) hide)
+    )
+    (property "Datasheet" "~" (at 205.74 73.025 0)
+      (effects (font (size 1.27 1.27)) hide)
+    )
+    (pin "1")
+    (pin "2")
+    (pin "3")
+    (pin "4")
+    (pin "5")
+    (pin "6")
+    (pin "7")
+    (pin "8")
+    (pin "9")
+    (instances
+      (project "motorgo_plink"
+        (path "/e63e39d7-6ac0-4ffd-8aa3-1841a4541b55/7d6efa12-7b94-467b-977c-f0e88b0f6fad"
+          (reference "J23") (unit 1)
+        )
+      )
+    )
+  )
   (symbol (lib_id "LCSC_imports:LIS3MDLTR") (at 83.185 73.66 0) (unit 1)
     (in_bom yes) (on_board yes) (dnp no) (fields_autoplaced)
@@
         (path "/e63e39d7-6ac0-4ffd-8aa3-1841a4541b55/7d6efa12-7b94-467b-977c-f0e88b0f6fad"
           (reference "U6") (unit 1)
+        )
+      )
+    )
+  )
+  (symbol (lib_id "power:+3V3") (at 141.605 88.265 0) (unit 1)
+    (in_bom yes) (on_board yes) (dnp no)
+    (property "Reference" "#PWR096" (at 141.605 92.075 0)
+      (effects (font (size 1.27 1.27)) hide)
+    )
+    (property "Value" "+3V3" (at 137.16 86.995 0)
+      (effects (font (size 1.27 1.27)))
+    )
+    (property "Footprint" "" (at 141.605 88.265 0)
+      (effects (font (size 1.27 1.27)) hide)
+    )
+    (property "Datasheet" "" (at 141.605 88.265 0)
+      (effects (font (size 1.27 1.27)) hide)
+    )
+    (pin "1")
+    (instances
+      (project "motorgo_plink"
+        (path "/e63e39d7-6ac0-4ffd-8aa3-1841a4541b55/7d6efa12-7b94-467b-977c-f0e88b0f6fad"
+          (reference "#PWR096") (unit 1)
         )
       )
@@
         )
       )
+    )
+  )
+  (symbol (lib_id "power:+3V3") (at 177.165 81.915 0) (unit 1)
+    (in_bom yes) (on_board yes) (dnp no) (fields_autoplaced)
+    (property "Reference" "#PWR0104" (at 177.165 85.725 0)
+      (effects (font (size 1.27 1.27)) hide)
+    )
+    (property "Value" "+3V3" (at 177.165 76.2 0)
+      (effects (font (size 1.27 1.27)))
+    )
+    (property "Footprint" "" (at 177.165 81.915 0)
+      (effects (font (size 1.27 1.27)) hide)
+    )
+    (property "Datasheet" "" (at 177.165 81.915 0)
+      (effects (font (size 1.27 1.27)) hide)
+    )
+    (pin "1")
+    (instances
+      (project "motorgo_plink"
+        (path "/e63e39d7-6ac0-4ffd-8aa3-1841a4541b55/7d6efa12-7b94-467b-977c-f0e88b0f6fad"
+          (reference "#PWR0104") (unit 1)
+        )
+      )

Commit message: WIP update, schematic mainly complete
Parts:
- added C16, C26: 100nF, symbol Device:C_Small
- added C27: 1uF, symbol Device:C_Polarized_Small
- added R18, R19, R26, R28, R34: 1k, symbol Device:R_Small
- added R27, R31, R37, R38, R39, R40, R41, R42: DNP, symbol Device:R_Small
- J23: symbol Connector:Conn_01x09_Pin -> Connector:Conn_01x06_Pin
Connections:
- net +3V3: now also U6.10 (CS), U6.5 (Vdd), U6.6 (Vdd_IO), C26.1, C27.1, R18.1, R19.1, R27.2, R31.2, R34.2
- net GND: now also U10.6 (GND), U10.7 (GND), U6.12 (Res), U6.2 (Res), U6.3 (GND), C16.1, C26.2, C27.2, R26.2, R28.2, R37.2, R38.2, R39.2, R40.2, R41.2, R42.2
- net INT1_acc: now reaches J23.1 (Pin_1)
- net INT1_acc: now also U10.4 (INT1), R37.1
- net INT2_acc: now reaches J23.2 (Pin_2)
- net INT2_acc: now also U10.9 (INT2), R38.1
- net SDO_acc: now reaches J23.3 (Pin_3)
- net SDO_acc: now also U10.1 (SDO/SA0), R28.1, R31.1, R39.1
- net DRDY_mag: now reaches J23.4 (Pin_4)
- net DRDY_mag: now also U6.8 (DRDY), R40.1
- net INT_mag: now reaches J23.5 (Pin_5)
- net INT_mag: now also U6.7 (INT), R41.1
- net SDO_mag: now reaches J23.6 (Pin_6)
- net SDO_mag: now also U6.9 (SD0/SA1), R26.1, R27.1, R42.1
- net SCL: now reaches U6.1 (SCL/SPC)
- net SCL: now also U10.14 (SDA), R19.2
- net SDA: now reaches U6.11 (SDA/SDI/SDO)
- net SDA: now also U10.13 (SCL), R18.2
- net at U6.4 (C1): now also C16.2
- net at U10.12 (CS): now also R34.1
- net SDX_acc: now reaches U10.2 (SDX)
- net SCX_acc: now reaches U10.3 (SCX)
- no-connect marks 0 -> 4
Other:
- note added: "LIS3MDLTR - 3 axis Gyroscope"
- note added: "LSM6DS3TR - 6 axis IMU"
- note added: "NOTE: The ground for these chips should be as seperate as possible from any sources of noise. The Magnetometer is esp sensitive to EMI"
- note added: "Pullup SCL and SDA lines"
- note added: "debugging breakout"
- note added: "for configuring SDO"
- moved on the sheet: U10, U6

Commit message: WIP update. Parts semi-finalized
Parts:
- C30: renamed from C16; footprint (none) -> Capacitor_SMD:C_01005_0402Metric
- C31: renamed from C26; footprint (none) -> Capacitor_SMD:C_01005_0402Metric
- C32: renamed from C27; footprint (none) -> Capacitor_SMD:C_0603_1608Metric
- J23: footprint (none) -> Connector_PinHeader_2.54mm:PinHeader_1x09_P2.54mm_Vertical
- R38: renamed from R18; value 1k -> 2k; footprint (none) -> Resistor_SMD:R_0402_1005Metric
- R39: renamed from R19; value 1k -> 2k; footprint (none) -> Resistor_SMD:R_0402_1005Metric
- R40: renamed from R37; footprint (none) -> Resistor_SMD:R_0402_1005Metric
- R41: renamed from R38; footprint (none) -> Resistor_SMD:R_0402_1005Metric
- R42: renamed from R39; footprint (none) -> Resistor_SMD:R_0402_1005Metric
- R43: renamed from R40; footprint (none) -> Resistor_SMD:R_0402_1005Metric
- R44: renamed from R41; footprint (none) -> Resistor_SMD:R_0402_1005Metric
- R45: renamed from R42; footprint (none) -> Resistor_SMD:R_0402_1005Metric
- R46: renamed from R26; footprint (none) -> Resistor_SMD:R_0402_1005Metric
- R47: renamed from R27; footprint (none) -> Resistor_SMD:R_0402_1005Metric
- R48: renamed from R31; footprint (none) -> Resistor_SMD:R_0402_1005Metric
- R49: renamed from R28; footprint (none) -> Resistor_SMD:R_0402_1005Metric
- R50: renamed from R34; footprint (none) -> Resistor_SMD:R_0402_1005Metric
- U10: renamed from U6; footprint kicad_lceda:LGA-12_L2.0-W2.0-P0.50-BL -> LCSC_parts:LIS3MDLTR_LGA-12
- U11: renamed from U10; footprint kicad_lceda:LGA-14_L3.0-W2.5-P0.50-TL -> LCSC_parts:LSM6DSOTR_LGA-14
Other:
- note added: "LIS3MDLTR - 3 axis Magnetometer"
- note removed: "LIS3MDLTR - 3 axis Gyroscope"

Commit message: WIP update. Layout begin
Parts:
- J23: value Conn_01x09_Pin -> Conn_01x06_Pin; footprint Connector_PinHeader_2.54mm:PinHeader_1x09_P2.54mm_Vertical -> Connector_PinHeader_1.00mm:PinHeader_1x06_P1.00mm_Vertical
Changed lines of the file:
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@@
       (effects (font (size 1.27 1.27)))
     )
-    (property "Value" "Conn_01x09_Pin" (at 126.365 48.26 0)
+    (property "Value" "Conn_01x06_Pin" (at 126.365 48.26 0)
       (effects (font (size 1.27 1.27)))
     )
-    (property "Footprint" "Connector_PinHeader_2.54mm:PinHeader_1x09_P2.54mm_Vertical" (at 114.3 57.15 0)
+    (property "Footprint" "Connector_PinHeader_1.00mm:PinHeader_1x06_P1.00mm_Vertical" (at 114.3 57.15 0)
       (effects (font (size 1.27 1.27)) hide)
     )

Commit message: WIP update. Ready for BOM editing
Parts:
- added R34: 0R0, symbol Device:R_Small
Connections:
- net GND: now also R34.2; no longer C30.1, C31.2, C32.2, R40.2, R41.2, R42.2, R43.2, R44.2, R45.2, R46.2, R49.2, U10.12 (Res), U10.2 (Res), U10.3 (GND), U11.6 (GND), U11.7 (GND)
- net +3V3 renamed +3.3V
- new net GNDD: C30.1, C31.2, C32.2, R34.1, R40.2, R41.2, R42.2, R43.2, R44.2, R45.2, R46.2, R49.2, U10.12 (Res), U10.2 (Res), U10.3 (GND), U11.6 (GND), U11.7 (GND)

Commit message: WIP update. change USBC port
Parts:
- R34: footprint (none) -> Resistor_SMD:R_0603_1608Metric
Changed lines of the file:
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@@
       (effects (font (size 1.27 1.27)))
     )
-    (property "Footprint" "" (at 238.125 70.485 0)
+    (property "Footprint" "Resistor_SMD:R_0603_1608Metric" (at 238.125 70.485 0)
       (effects (font (size 1.27 1.27)) hide)
     )

Commit message: WIP (TS) - updating BOM with values from other branch.
Parts:
- C30, C31: footprint Capacitor_SMD:C_01005_0402Metric -> Capacitor_SMD:C_0402_1005Metric; Field4 (none) -> CHANGED FOOTPRINT 6-3-24; LCSC_Part_Number (none) -> C880603
- C32: LCSC_Part_Number (none) -> C15849
Changed lines of the file:
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@@
       (effects (font (size 1.27 1.27)))
     )
-    (property "Footprint" "Capacitor_SMD:C_01005_0402Metric" (at 59.055 118.745 0)
-      (effects (font (size 1.27 1.27)) hide)
-    )
-    (property "Datasheet" "~" (at 59.055 118.745 0)
+    (property "Footprint" "Capacitor_SMD:C_0402_1005Metric" (at 59.055 118.745 0)
+      (effects (font (size 1.27 1.27)) hide)
+    )
+    (property "Datasheet" "https://www.lcsc.com/product-detail/Multilayer-Ceramic-Capacitors-MLCC-SMD-SMT_CCTC-TCC0402X5R104K250AT_C880603.html" (at 59.055 118.745 0)
+      (effects (font (size 1.27 1.27)) hide)
+    )
+    (property "Field4" "CHANGED FOOTPRINT 6-3-24" (at 59.055 118.745 0)
+      (effects (font (size 1.27 1.27)) hide)
+    )
+    (property "LCSC_Part_Number" "C880603" (at 59.055 118.745 0)
       (effects (font (size 1.27 1.27)) hide)
     )
@@
       (effects (font (size 1.27 1.27)))
     )
-    (property "Footprint" "Capacitor_SMD:C_01005_0402Metric" (at 76.835 119.38 0)
-      (effects (font (size 1.27 1.27)) hide)
-    )
-    (property "Datasheet" "~" (at 76.835 119.38 0)
+    (property "Footprint" "Capacitor_SMD:C_0402_1005Metric" (at 76.835 119.38 0)
+      (effects (font (size 1.27 1.27)) hide)
+    )
+    (property "Datasheet" "https://www.lcsc.com/product-detail/Multilayer-Ceramic-Capacitors-MLCC-SMD-SMT_CCTC-TCC0402X5R104K250AT_C880603.html" (at 76.835 119.38 0)
+      (effects (font (size 1.27 1.27)) hide)
+    )
+    (property "Field4" "CHANGED FOOTPRINT 6-3-24" (at 76.835 119.38 0)
+      (effects (font (size 1.27 1.27)) hide)
+    )
+    (property "LCSC_Part_Number" "C880603" (at 76.835 119.38 0)
       (effects (font (size 1.27 1.27)) hide)
     )
@@
       (effects (font (size 1.27 1.27)) hide)
     )
-    (property "Datasheet" "~" (at 82.55 119.38 0)
-      (effects (font (size 1.27 1.27)) hide)
-    )
+    (property "Datasheet" "https://www.lcsc.com/product-detail/Multilayer-Ceramic-Capacitors-MLCC-SMD-SMT_Samsung-Electro-Mechanics-CL10A105KB8NNNC_C15849.html" (at 82.55 119.38 0)
+      (effects (font (size 1.27 1.27)) hide)
+    )
+    (property "LCSC_Part_Number" "C15849" (at 82.55 119.38 0)
+      (effects (font (size 1.27 1.27)) hide)
+    )

Commit message: updated BOM in prep for order - TS
Parts:
- J23: Field4 (none) -> only 1 option, only 10 in stock. DNP?; LCSC_Part_Number (none) -> C7434639
- R34: LCSC_Part_Number (none) -> C2906858
- R38, R39: LCSC_Part_Number (none) -> C4109
- R46, R49, R50: LCSC_Part_Number (none) -> C2906899
- U10: LCSC_Part_Number (none) -> C478483
- U11: LCSC_Part_Number (none) -> C95230
Changed lines of the file:
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@@
       (effects (font (size 1.27 1.27)) hide)
     )
-    (property "Datasheet" "~" (at 71.12 57.785 0)
+    (property "Datasheet" "https://www.lcsc.com/product-detail/Chip-Resistor-Surface-Mount_UNI-ROYAL-Uniroyal-Elec-0402WGF2001TCE_C4109.html" (at 71.12 57.785 0)
+      (effects (font (size 1.27 1.27)) hide)
+    )
+    (property "LCSC_Part_Number" "C4109" (at 71.12 57.785 0)
       (effects (font (size 1.27 1.27)) hide)
     )
@@
       (effects (font (size 1.27 1.27)) hide)
     )
-    (property "Datasheet" "~" (at 175.26 123.825 0)
+    (property "Datasheet" "https://www.lcsc.com/product-detail/Chip-Resistor-Surface-Mount_FOJAN-FRC0402J102-TS_C2906899.html" (at 175.26 123.825 0)
+      (effects (font (size 1.27 1.27)) hide)
+    )
+    (property "LCSC_Part_Number" "C2906899" (at 175.26 123.825 0)
       (effects (font (size 1.27 1.27)) hide)
     )
@@
       (effects (font (size 1.27 1.27)) hide)
     )
-    (property "Datasheet" "~" (at 146.685 123.825 0)
+    (property "Datasheet" "https://www.lcsc.com/product-detail/Chip-Resistor-Surface-Mount_FOJAN-FRC0402J102-TS_C2906899.html" (at 146.685 123.825 0)
+      (effects (font (size 1.27 1.27)) hide)
+    )
+    (property "LCSC_Part_Number" "C2906899" (at 146.685 123.825 0)
       (effects (font (size 1.27 1.27)) hide)
     )
@@
       (effects (font (size 1.27 1.27)) hide)
     )
-    (property "Datasheet" "~" (at 114.3 57.15 0)
+    (property "Datasheet" "https://www.lcsc.com/product-detail/Pin-Headers_GREENCONN-GPCD101-0602A003C1AH_C7434639.html" (at 114.3 57.15 0)
+      (effects (font (size 1.27 1.27)) hide)
+    )
+    (property "Field4" "only 1 option, only 10 in stock. DNP?" (at 114.3 57.15 0)
+      (effects (font (size 1.27 1.27)) hide)
+    )
+    (property "LCSC_Part_Number" "C7434639" (at 114.3 57.15 0)
       (effects (font (size 1.27 1.27)) hide)
     )
@@
       (effects (font (size 1.27 1.27)) hide)
     )
-    (property "Datasheet" "~" (at 238.125 70.485 0)
+    (property "Datasheet" "https://www.lcsc.com/product-detail/Chip-Resistor-Surface-Mount_FOJAN-FRC0402F0000TS_C2906858.html" (at 238.125 70.485 0)
+      (effects (font (size 1.27 1.27)) hide)
+    )
+    (property "LCSC_Part_Number" "C2906858" (at 238.125 70.485 0)
       (effects (font (size 1.27 1.27)) hide)
     )
@@
       (effects (font (size 1.27 1.27)) hide)
     )
-    (property "Datasheet" "http://www.szlcsc.com/product/details_485763.html" (at 110.49 85.0138 0)
+    (property "Datasheet" "https://www.lcsc.com/product-detail/Linear-Hall-Sensors_STMicroelectronics-LIS3MDLTR_C478483.html" (at 110.49 85.0138 0)
       (effects (font (size 1.27 1.27)) hide)
     )
@@
     )
     (property "uuid" "std:3c4a1927816047c0b32d8307cf40d91b" (at 110.49 88.1888 0)
+      (effects (font (size 1.27 1.27)) hide)
+    )
+    (property "LCSC_Part_Number" "C478483" (at 111.125 104.14 0)
       (effects (font (size 1.27 1.27)) hide)
     )
@@
       (effects (font (size 1.27 1.27)) hide)
     )
-    (property "Datasheet" "~" (at 76.2 57.785 0)
+    (property "Datasheet" "https://www.lcsc.com/product-detail/Chip-Resistor-Surface-Mount_UNI-ROYAL-Uniroyal-Elec-0402WGF2001TCE_C4109.html" (at 76.2 57.785 0)
+      (effects (font (size 1.27 1.27)) hide)
+    )
+    (property "LCSC_Part_Number" "C4109" (at 76.2 57.785 0)
       (effects (font (size 1.27 1.27)) hide)
     )
@@
       (effects (font (size 1.27 1.27)) hide)
     )
-    (property "Datasheet" "~" (at 227.965 92.075 0)
+    (property "Datasheet" "https://www.lcsc.com/product-detail/Chip-Resistor-Surface-Mount_FOJAN-FRC0402J102-TS_C2906899.html" (at 227.965 92.075 0)
+      (effects (font (size 1.27 1.27)) hide)
+    )
+    (property "LCSC_Part_Number" "C2906899" (at 227.965 92.075 0)
       (effects (font (size 1.27 1.27)) hide)
     )
@@
       (effects (font (size 1.27 1.27)) hide)
     )
-    (property "Datasheet" "http://www.szlcsc.com/product/details_96431.html" (at 211.455 103.5558 0)
+    (property "Datasheet" "https://www.lcsc.com/product-detail/Attitude-Sensor-Gyroscope_STMicroelectronics-LSM6DS3TR_C95230.html" (at 211.455 103.5558 0)
       (effects (font (size 1.27 1.27)) hide)
     )
@@
       (effects (font (size 1.27 1.27)) hide)
     )
+    (property "LCSC_Part_Number" "C95230" (at 211.455 109.22 0)
+      (effects (font (size 1.27 1.27)) hide)
+    )
