File: motorgo_plink/motor_go_power_system.kicad_sch (KiCad schematic)
At the start: 21 parts, among them U11 HUSB238_002DD, U7 AMS1117-3.3, U9 TPS54620RHLR

Commit message: WIP update, schematic mainly complete
Parts:
- added C28: 1uF, symbol Device:C_Small
- added J11: USB4520-03-0-A_REVA, aaa_motorgo_components:GCT_USB4520-03-0-A_REVA, symbol USB4520-03-0-A_REVA:USB4520-03-0-A_REVA
- added JP4: SolderJumper_2_Bridged, symbol Jumper:SolderJumper_2_Bridged
- added JP5, JP6: SolderJumper_2_Open, symbol Jumper:SolderJumper_2_Open
- added Q1: SI2323, symbol Device:Q_PMOS_GSD
- added R43: 10K, symbol Device:R_US
- added R44: 10.5K, symbol Device:R_US
- added R45: 14K, symbol Device:R_US
- added R46: 10R 1%, symbol Device:R_US
- added R47: 49.9K, symbol Device:R_US
- added R48: 5.1K, symbol Device:R_US
Connections:
- net +BATT: now also Q1.3 (D)
- net GND: now also C28.2, J11.A1_B12 (GND_A), J11.B1_A12 (GND_B), J11.S1 (SHELL_GND), J11.S2 (SHELL_GND), J11.S3 (SHELL_GND), J11.S4 (SHELL_GND), R43.2, R44.2, R45.2
- net at U11.1 (VIN): now also C28.1, R46.2
- net at U11.10 (GATE): now also R48.1
- net CC1: now reaches U11.4 (CC1)
- net CC1: now also J11.A5 (CC1)
- net CC2: now reaches U11.5 (CC2)
- net CC2: now also J11.B5 (CC2)
- net sda_pd: now reaches U11.6 (SDA)
- net scl_pd: now reaches U11.7 (SCL)
- net at U11.8 (VSET): now also JP4.2 (B), JP5.2 (B)
- net at U11.9 (ISET): now also JP6.2 (B)
- new net: JP6.1 (A), R44.1
- new net: Q1.1 (G), R47.2, R48.2
- new net: JP4.1 (A), R43.1
- new net: JP5.1 (A), R45.1
- new net +VDC: J11.A4_B9 (VBUS_A), J11.B4_A9 (VBUS_B), Q1.2 (S), R46.1, R47.1
- no-connect marks 1 -> 9
Other:
- note added: "10K 12V 14K 15V Hiz 20V"
- note added: "Hiz 3.25A 10.5K 2.00A"
- note added: "Imax select"
- note added: "R Iset"
- note added: "R Vset"
- note added: "USBC Power Input"
- note added: "Vmax select"
- moved on the sheet: C10, C12, C13, C9, R10, R11, R12, R13, U11, U9

Commit message: WIP update. Parts semi-finalized
Parts:
- added R18, R19: DNP, Resistor_SMD:R_0402_1005Metric, symbol Device:R_Small
- C15: renamed from C9; footprint (none) -> Capacitor_SMD:C_0805_2012Metric
- C17: renamed from C10; footprint (none) -> Capacitor_SMD:C_0603_1608Metric
- C18: renamed from C12; footprint (none) -> Capacitor_SMD:C_0201_0603Metric
- C20: renamed from C13; footprint (none) -> Capacitor_SMD:C_0201_0603Metric
- C21: renamed from C28; footprint (none) -> Capacitor_SMD:C_0603_1608Metric
- C22: renamed from C14; footprint (none) -> Capacitor_SMD:C_0402_1005Metric
- C23: renamed from C15; footprint (none) -> Capacitor_SMD:C_1210_3225Metric
- J11: footprint aaa_motorgo_components:GCT_USB4520-03-0-A_REVA -> mg_mini_v1r3:GCT_USB4520-03-0-A_REVA
- J8: footprint aaa_motorgo_components:xt30 -> LCSC_parts:CONN-TH_DC-005-2.5A-2.0
- JP4: footprint (none) -> Jumper:SolderJumper-2_P1.3mm_Bridged2Bar_RoundedPad1.0x1.5mm
- JP5, JP6: footprint (none) -> Jumper:SolderJumper-2_P1.3mm_Open_RoundedPad1.0x1.5mm
- L1: footprint (none) -> LCSC_parts:IND-SMD_L7.3-W6.6
- Q1: footprint (none) -> LCSC_parts:SI2323_SOT-23-3_L2.9-W1.3-P0.95-LS2.4-BR
- R16: renamed from R10; footprint (none) -> Resistor_SMD:R_0402_1005Metric
- R17: renamed from R11; footprint (none) -> Resistor_SMD:R_0402_1005Metric
- R18: renamed from R12; footprint (none) -> Resistor_SMD:R_0402_1005Metric
- R19: renamed from R13; footprint (none) -> Resistor_SMD:R_0402_1005Metric
- R20: renamed from R46; footprint (none) -> Resistor_SMD:R_0402_1005Metric
- R23: renamed from R48; footprint (none) -> Resistor_SMD:R_0402_1005Metric
- R24: renamed from R16; footprint (none) -> Resistor_SMD:R_0402_1005Metric
- R25: renamed from R17; footprint (none) -> Resistor_SMD:R_0402_1005Metric
- R26: renamed from R47; footprint (none) -> Resistor_SMD:R_0402_1005Metric
- R27: renamed from R43; footprint (none) -> Resistor_SMD:R_0402_1005Metric
- R28: renamed from R45; footprint (none) -> Resistor_SMD:R_0402_1005Metric
- R29: renamed from R44; footprint (none) -> Resistor_SMD:R_0402_1005Metric
- U6: renamed from U9; footprint kicad_lceda:VQFN-14_L3.5-W3.5-P0.50-TL-EP_TPS54622RHLT -> LCSC_parts:VQFN-14_L3.5-W3.5-P0.50-TL-EP_TPS54622RHLT
- U7: renamed from U11; footprint kicad_lceda:DFN-10_L3.0-W3.0-P0.50-BL-EP2.5 -> LCSC_parts:DFN-10_L3.0-W3.0-P0.50-BL-EP2.5
- renumbered C11 to C16, C39 to C19, C17 to C24, C29 to C25, U7 to U8
Connections:
- net scl_pd: now also R19.2
- net sda_pd: now also R18.2
- new net +3V3: R18.1, R19.1
Other:
- note added: "i2c pullup"
- moved on the sheet: JP4, JP5, JP6, R27, R28, R29

Commit message: WIP update. Layout begin
Parts:
- removed C19: 220uF 50v, Capacitor_SMD:CP_Elec_10x10, symbol motorgo_components:RGA221M1EBK-0811G
Other:
- moved on the sheet: C16
Changed lines of the file:
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@@
 (kicad_sch (version 20230121) (generator eeschema)
   (paper "A4")
+  (junction (at 56.515 140.335) (diameter 0) (color 0 0 0 0)
+  )
+  (junction (at 113.03 65.405) (diameter 0) (color 0 0 0 0)
+  )
+  (junction (at 43.815 70.485) (diameter 0) (color 0 0 0 0)
+  )
+  (junction (at 167.64 62.23) (diameter 0) (color 0 0 0 0)
+  )
+  (junction (at 206.375 59.055) (diameter 0) (color 0 0 0 0)
+  )
+  (junction (at 184.785 59.055) (diameter 0) (color 0 0 0 0)
+  )
+  (junction (at 195.58 74.295) (diameter 0) (color 0 0 0 0)
+  )
+  (junction (at 80.645 70.485) (diameter 0) (color 0 0 0 0)
+  )
+  (junction (at 123.825 65.405) (diameter 0) (color 0 0 0 0)
+  )
+  (junction (at 56.515 109.855) (diameter 0) (color 0 0 0 0)
+  )
+  (junction (at 156.845 65.405) (diameter 0) (color 0 0 0 0)
+  )
+  (junction (at 214.63 97.79) (diameter 0) (color 0 0 0 0)
+  )
+  (junction (at 142.875 94.615) (diameter 0) (color 0 0 0 0)
+  )
+  (junction (at 104.775 140.97) (diameter 0) (color 0 0 0 0)
+  )
+  (junction (at 200.025 149.225) (diameter 0) (color 0 0 0 0)
+  )
+  (junction (at 194.945 149.225) (diameter 0) (color 0 0 0 0)
+  )
+  (junction (at 145.415 140.97) (diameter 0) (color 0 0 0 0)
+  )
+  (junction (at 53.975 153.035) (diameter 0) (color 0 0 0 0)
+  )
+  (junction (at 113.03 93.345) (diameter 0) (color 0 0 0 0)
+  )
+  (junction (at 148.59 175.26) (diameter 0) (color 0 0 0 0)
+  )
+  (junction (at 142.875 65.405) (diameter 0) (color 0 0 0 0)
+  )
+  (junction (at 55.245 70.485) (diameter 0) (color 0 0 0 0)
+  )
+  (junction (at 142.875 78.105) (diameter 0) (color 0 0 0 0)
+  )
+  (junction (at 217.805 97.79) (diameter 0) (color 0 0 0 0)
+  )
+  (junction (at 60.96 70.485) (diameter 0) (color 0 0 0 0)
+  )
   (junction (at 56.515 153.035) (diameter 0) (color 0 0 0 0)
   )
-  (junction (at 113.03 65.405) (diameter 0) (color 0 0 0 0)
-  )
-  (junction (at 43.815 70.485) (diameter 0) (color 0 0 0 0)
-  )
-  (junction (at 167.64 62.23) (diameter 0) (color 0 0 0 0)
-  )
-  (junction (at 206.375 59.055) (diameter 0) (color 0 0 0 0)
-  )
-  (junction (at 184.785 59.055) (diameter 0) (color 0 0 0 0)
-  )
-  (junction (at 195.58 74.295) (diameter 0) (color 0 0 0 0)
-  )
-  (junction (at 80.645 70.485) (diameter 0) (color 0 0 0 0)
-  )
-  (junction (at 123.825 65.405) (diameter 0) (color 0 0 0 0)
-  )
-  (junction (at 56.515 109.855) (diameter 0) (color 0 0 0 0)
-  )
-  (junction (at 156.845 65.405) (diameter 0) (color 0 0 0 0)
-  )
-  (junction (at 214.63 97.79) (diameter 0) (color 0 0 0 0)
-  )
-  (junction (at 142.875 94.615) (diameter 0) (color 0 0 0 0)
-  )
-  (junction (at 104.775 140.97) (diameter 0) (color 0 0 0 0)
-  )
-  (junction (at 200.025 149.225) (diameter 0) (color 0 0 0 0)
-  )
-  (junction (at 194.945 149.225) (diameter 0) (color 0 0 0 0)
-  )
-  (junction (at 145.415 140.97) (diameter 0) (color 0 0 0 0)
-  )
-  (junction (at 53.975 153.035) (diameter 0) (color 0 0 0 0)
-  )
-  (junction (at 113.03 93.345) (diameter 0) (color 0 0 0 0)
-  )
-  (junction (at 148.59 175.26) (diameter 0) (color 0 0 0 0)
-  )
-  (junction (at 142.875 65.405) (diameter 0) (color 0 0 0 0)
-  )
-  (junction (at 55.245 70.485) (diameter 0) (color 0 0 0 0)
-  )
-  (junction (at 142.875 78.105) (diameter 0) (color 0 0 0 0)
-  )
-  (junction (at 217.805 97.79) (diameter 0) (color 0 0 0 0)
-  )
-  (junction (at 60.96 70.485) (diameter 0) (color 0 0 0 0)
-  )
   (junction (at 197.485 152.4) (diameter 0) (color 0 0 0 0)
   )
@@
   )
   (junction (at 198.755 149.225) (diameter 0) (color 0 0 0 0)
-  )
-  (junction (at 56.515 140.335) (diameter 0) (color 0 0 0 0)
   )
   (junction (at 53.975 140.335) (diameter 0) (color 0 0 0 0)
@@
     (stroke (width 0) (type default))
   )
-  (wire (pts (xy 56.515 140.335) (xy 69.215 140.335))
-    (stroke (width 0) (type default))
-  )
   (wire (pts (xy 113.03 93.345) (xy 113.03 109.22))
     (stroke (width 0) (type default))
@@
   )
   (wire (pts (xy 206.375 59.055) (xy 208.915 59.055))
-    (stroke (width 0) (type default))
-  )
-  (wire (pts (xy 56.515 153.035) (xy 69.215 153.035))
     (stroke (width 0) (type default))
   )
@@
     )
   )
-  (symbol (lib_id "motorgo_components:RGA221M1EBK-0811G") (at 53.975 140.335 270) (unit 1)
+  (symbol (lib_id "motorgo_components:RGA221M1EBK-0811G") (at 56.515 140.335 270) (unit 1)
     (in_bom yes) (on_board yes) (dnp no) (fields_autoplaced)
-    (property "Reference" "C16" (at 57.785 146.05 90)
-      (effects (font (size 1.27 1.27)) (justify left))
-    )
-    (property "Value" "220uF 50v" (at 57.785 148.59 90)
-      (effects (font (size 1.27 1.27)) (justify left))
-    )
-    (property "Footprint" "Capacitor_SMD:CP_Elec_10x10" (at -42.215 149.225 0)
-      (effects (font (size 1.27 1.27)) (justify left top) hide)
-    )
-    (property "Datasheet" "https://datasheet.lcsc.com/lcsc/2304140030_Nichicon-UWT1H221MNL1GS_C125977.pdf" (at -142.215 149.225 0)
-      (effects (font (size 1.27 1.27)) (justify left top) hide)
-    )
-    (property "Height" "13" (at -342.215 149.225 0)
-      (effects (font (size 1.27 1.27)) (justify left top) hide)
-    )
-    (property "Mouser Part Number" "140-RGA221M1EBK0811G" (at -442.215 149.225 0)
-      (effects (font (size 1.27 1.27)) (justify left top) hide)
-    )
-    (property "Mouser Price/Stock" "https://www.mouser.co.uk/ProductDetail/Lelon/RGA221M1EBK-0811G?qs=pNDdEcSXiOD075vn7PGSsQ%3D%3D" (at -542.215 149.225 0)
-      (effects (font (size 1.27 1.27)) (justify left top) hide)
-    )
-    (property "Manufacturer_Name" "Lelon" (at -642.215 149.225 0)
-      (effects (font (size 1.27 1.27)) (justify left top) hide)
-    )
-    (property "Manufacturer_Part_Number" "RGA221M1EBK-0811G" (at -742.215 149.225 0)
-      (effects (font (size 1.27 1.27)) (justify left top) hide)
-    )
-    (property "LCSC_Part_Number" "C125977" (at 53.975 140.335 0)
+    (property "Reference" "C16" (at 60.325 146.05 90)
+      (effects (font (size 1.27 1.27)) (justify left))
+    )
+    (property "Value" "220uF 50v" (at 60.325 148.59 90)
+      (effects (font (size 1.27 1.27)) (justify left))
+    )
+    (property "Footprint" "Capacitor_SMD:CP_Elec_10x10" (at -39.675 149.225 0)
+      (effects (font (size 1.27 1.27)) (justify left top) hide)
+    )
+    (property "Datasheet" "https://datasheet.lcsc.com/lcsc/2304140030_Nichicon-UWT1H221MNL1GS_C125977.pdf" (at -139.675 149.225 0)
+      (effects (font (size 1.27 1.27)) (justify left top) hide)
+    )
+    (property "Height" "13" (at -339.675 149.225 0)
+      (effects (font (size 1.27 1.27)) (justify left top) hide)
+    )
+    (property "Mouser Part Number" "140-RGA221M1EBK0811G" (at -439.675 149.225 0)
+      (effects (font (size 1.27 1.27)) (justify left top) hide)
+    )
+    (property "Mouser Price/Stock" "https://www.mouser.co.uk/ProductDetail/Lelon/RGA221M1EBK-0811G?qs=pNDdEcSXiOD075vn7PGSsQ%3D%3D" (at -539.675 149.225 0)
+      (effects (font (size 1.27 1.27)) (justify left top) hide)
+    )
+    (property "Manufacturer_Name" "Lelon" (at -639.675 149.225 0)
+      (effects (font (size 1.27 1.27)) (justify left top) hide)
+    )
+    (property "Manufacturer_Part_Number" "RGA221M1EBK-0811G" (at -739.675 149.225 0)
+      (effects (font (size 1.27 1.27)) (justify left top) hide)
+    )
+    (property "LCSC_Part_Number" "C125977" (at 56.515 140.335 0)
       (effects (font (size 1.27 1.27)) hide)
     )
@@
         )
       )
-    )
-  )
-  (symbol (lib_id "motorgo_components:RGA221M1EBK-0811G") (at 69.215 140.335 270) (unit 1)
-    (in_bom yes) (on_board yes) (dnp no) (fields_autoplaced)
-    (property "Reference" "C19" (at 73.025 146.05 90)
-      (effects (font (size 1.27 1.27)) (justify left))
-    )
-    (property "Value" "220uF 50v" (at 73.025 148.59 90)
-      (effects (font (size 1.27 1.27)) (justify left))
-    )
-    (property "Footprint" "Capacitor_SMD:CP_Elec_10x10" (at -26.975 149.225 0)
-      (effects (font (size 1.27 1.27)) (justify left top) hide)
-    )
-    (property "Datasheet" "https://datasheet.lcsc.com/lcsc/2304140030_Nichicon-UWT1H221MNL1GS_C125977.pdf" (at -126.975 149.225 0)
-      (effects (font (size 1.27 1.27)) (justify left top) hide)
-    )
-    (property "Height" "13" (at -326.975 149.225 0)
-      (effects (font (size 1.27 1.27)) (justify left top) hide)
-    )
-    (property "Mouser Part Number" "140-RGA221M1EBK0811G" (at -426.975 149.225 0)
-      (effects (font (size 1.27 1.27)) (justify left top) hide)
-    )
-    (property "Mouser Price/Stock" "https://www.mouser.co.uk/ProductDetail/Lelon/RGA221M1EBK-0811G?qs=pNDdEcSXiOD075vn7PGSsQ%3D%3D" (at -526.975 149.225 0)
-      (effects (font (size 1.27 1.27)) (justify left top) hide)
-    )
-    (property "Manufacturer_Name" "Lelon" (at -626.975 149.225 0)
-      (effects (font (size 1.27 1.27)) (justify left top) hide)
-    )
-    (property "Manufacturer_Part_Number" "RGA221M1EBK-0811G" (at -726.975 149.225 0)
-      (effects (font (size 1.27 1.27)) (justify left top) hide)
-    )
-    (property "LCSC_Part_Number" "C125977" (at 69.215 140.335 0)
-      (effects (font (size 1.27 1.27)) hide)
-    )
-    (pin "1")
-    (pin "2")
-    (instances
-      (project "motorgo_plink"
-        (path "/e63e39d7-6ac0-4ffd-8aa3-1841a4541b55/c5a81061-28ff-4599-a380-43adb8d460db"
-          (reference "C19") (unit 1)
-        )
-      )

Commit message: WIP update. Ready for BOM editing
Parts:
- C24: value 22uF 10v -> 22uF 16v; footprint Capacitor_SMD:C_0402_1005Metric -> Capacitor_SMD:C_0603_1608Metric
Connections:
- net +3V3 is gone; now on net +3.3V: R18.1, R19.1
- net GND: now also U6.15 (EP)
Changed lines of the file:
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@@
 (kicad_sch (version 20230121) (generator eeschema)
   (paper "A4")
+  (junction (at 113.03 90.805) (diameter 0) (color 0 0 0 0)
+  )
   (junction (at 56.515 140.335) (diameter 0) (color 0 0 0 0)
   )
@@
     (stroke (width 0) (type default))
   )
+  (wire (pts (xy 113.03 90.805) (xy 113.03 93.345))
+    (stroke (width 0) (type default))
+  )
   (wire (pts (xy 132.08 151.13) (xy 130.175 151.13))
     (stroke (width 0) (type default))
@@
     (stroke (width 0) (type default))
   )
-  (wire (pts (xy 113.03 90.805) (xy 113.03 93.345))
+  (wire (pts (xy 113.03 88.265) (xy 113.03 90.805))
     (stroke (width 0) (type default))
   )
@@
       (effects (font (size 1.27 1.27)) (justify left))
     )
-    (property "Value" "22uF 10v" (at 177.8 64.77 90)
-      (effects (font (size 1.27 1.27)) (justify left))
-    )
-    (property "Footprint" "Capacitor_SMD:C_0402_1005Metric" (at 88.595 69.215 0)
+    (property "Value" "22uF 16v" (at 177.8 64.77 90)
+      (effects (font (size 1.27 1.27)) (justify left))
+    )
+    (property "Footprint" "Capacitor_SMD:C_0603_1608Metric" (at 88.595 69.215 0)
       (effects (font (size 1.27 1.27)) (justify left top) hide)
     )
@@
         (path "/e63e39d7-6ac0-4ffd-8aa3-1841a4541b55/c5a81061-28ff-4599-a380-43adb8d460db"
           (reference "#FLG02") (unit 1)
+        )
+      )
+    )
+  )
+  (symbol (lib_id "power:+3.3V") (at 206.375 57.15 0) (unit 1)
+    (in_bom yes) (on_board yes) (dnp no) (fields_autoplaced)
+    (property "Reference" "#PWR075" (at 206.375 60.96 0)
+      (effects (font (size 1.27 1.27)) hide)
+    )
+    (property "Value" "+3.3V" (at 206.375 52.07 0)
+      (effects (font (size 1.27 1.27)))
+    )
+    (property "Footprint" "" (at 206.375 57.15 0)
+      (effects (font (size 1.27 1.27)) hide)
+    )
+    (property "Datasheet" "" (at 206.375 57.15 0)
+      (effects (font (size 1.27 1.27)) hide)
+    )
+    (pin "1")
+    (instances
+      (project "motorgo_plink"
+        (path "/e63e39d7-6ac0-4ffd-8aa3-1841a4541b55/c5a81061-28ff-4599-a380-43adb8d460db"
+          (reference "#PWR075") (unit 1)
         )
       )
@@
         (path "/e63e39d7-6ac0-4ffd-8aa3-1841a4541b55/c5a81061-28ff-4599-a380-43adb8d460db"
           (reference "Q1") (unit 1)
-        )
-      )
-    )
-  )
-  (symbol (lib_id "power:+3V3") (at 109.22 165.735 0) (unit 1)
-    (in_bom yes) (on_board yes) (dnp no)
-    (property "Reference" "#PWR0108" (at 109.22 169.545 0)
-      (effects (font (size 1.27 1.27)) hide)
-    )
-    (property "Value" "+3V3" (at 113.03 163.83 0)
-      (effects (font (size 1.27 1.27)))
-    )
-    (property "Footprint" "" (at 109.22 165.735 0)
-      (effects (font (size 1.27 1.27)) hide)
-    )
-    (property "Datasheet" "" (at 109.22 165.735 0)
-      (effects (font (size 1.27 1.27)) hide)
-    )
-    (pin "1")
-    (instances
-      (project "motorgo_plink"
-        (path "/e63e39d7-6ac0-4ffd-8aa3-1841a4541b55/7d6efa12-7b94-467b-977c-f0e88b0f6fad"
-          (reference "#PWR0108") (unit 1)
-        )
-        (path "/e63e39d7-6ac0-4ffd-8aa3-1841a4541b55/c5a81061-28ff-4599-a380-43adb8d460db"
-          (reference "#PWR064") (unit 1)
         )
       )
@@
     )
   )
-  (symbol (lib_id "power:+3.3V") (at 206.375 57.15 0) (unit 1)
-    (in_bom yes) (on_board yes) (dnp no) (fields_autoplaced)
-    (property "Reference" "#PWR075" (at 206.375 60.96 0)
-      (effects (font (size 1.27 1.27)) hide)
-    )
-    (property "Value" "+3.3V" (at 206.375 53.34 0)
-      (effects (font (size 1.27 1.27)))
-    )
-    (property "Footprint" "" (at 206.375 57.15 0)
-      (effects (font (size 1.27 1.27)) hide)
-    )
-    (property "Datasheet" "" (at 206.375 57.15 0)
-      (effects (font (size 1.27 1.27)) hide)
-    )
-    (pin "1")
-    (instances
-      (project "motorgo_plink"
-        (path "/e63e39d7-6ac0-4ffd-8aa3-1841a4541b55/c5a81061-28ff-4599-a380-43adb8d460db"
-          (reference "#PWR075") (unit 1)
-        )
-      )
-    )
-  )
   (symbol (lib_id "power:GND") (at 148.59 175.26 0) (unit 1)
     (in_bom yes) (on_board yes) (dnp no) (fields_autoplaced)
@@
         )
       )
+    )
+  )
+  (symbol (lib_id "power:+3.3V") (at 109.22 165.735 0) (unit 1)
+    (in_bom yes) (on_board yes) (dnp no)
+    (property "Reference" "#PWR0118" (at 109.22 169.545 0)
+      (effects (font (size 1.27 1.27)) hide)
+    )
+    (property "Value" "+3.3V" (at 113.03 165.1 0)
+      (effects (font (size 1.27 1.27)))
+    )
+    (property "Footprint" "" (at 109.22 165.735 0)
+      (effects (font (size 1.27 1.27)) hide)
+    )
+    (property "Datasheet" "" (at 109.22 165.735 0)
+      (effects (font (size 1.27 1.27)) hide)
+    )
+    (pin "1")
+    (instances
+      (project "motorgo_plink"
+        (path "/e63e39d7-6ac0-4ffd-8aa3-1841a4541b55/c5a81061-28ff-4599-a380-43adb8d460db"
+          (reference "#PWR0118") (unit 1)
+        )
+      )
