File: motorgo_plink/motor_go_power_system.kicad_sch (KiCad schematic)
At the start: 34 parts, among them J11 USB4520-03-0-A_REVA, Q1 SI2323, U6 TPS54620RHLR, U7 HUSB238_002DD, U8 AMS1117-3.3

Commit message: WIP - adding P/Ns to BOM (TS). will finish in afternoon.
Parts:
- C15: LCSC_Part_Number (none) -> C5448891
- C17: LCSC_Part_Number (none) -> C6119856
- C18: LCSC_Part_Number (none) -> C285033
- C20: LCSC_Part_Number (none) -> C3037638
- C21: LCSC_Part_Number (none) -> C15849
- C22: LCSC_Part_Number (none) -> C880603
- C23: LCSC_Part_Number (none) -> C7432791
- C24: LCSC_Part_Number C3845593 -> C2762594
Changed lines of the file:
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@@
       (effects (font (size 1.27 1.27)) (justify left top) hide)
     )
-    (property "Datasheet" "https://datasheet.lcsc.com/lcsc/2308111745_Murata-Electronics-GRM158R61A226ME15D_C3845593.pdf" (at -11.405 69.215 0)
+    (property "Datasheet" "https://www.lcsc.com/product-detail/Multilayer-Ceramic-Capacitors-MLCC-SMD-SMT_Samsung-Electro-Mechanics-CL10A226MO7JZNC_C2762594.html" (at -11.405 69.215 0)
       (effects (font (size 1.27 1.27)) (justify left top) hide)
     )
@@
       (effects (font (size 1.27 1.27)) (justify left top) hide)
     )
-    (property "LCSC_Part_Number" "C3845593" (at 184.785 60.325 0)
+    (property "LCSC_Part_Number" "C2762594" (at 184.785 60.325 0)
       (effects (font (size 1.27 1.27)) hide)
     )
@@
       (effects (font (size 1.27 1.27)) hide)
     )
-    (property "Datasheet" "~" (at 156.845 78.74 0)
+    (property "Datasheet" "https://www.lcsc.com/product-detail/Multilayer-Ceramic-Capacitors-MLCC-SMD-SMT_Chinocera-HGC1210R5476M250NSVK_C7432791.html" (at 156.845 78.74 0)
+      (effects (font (size 1.27 1.27)) hide)
+    )
+    (property "LCSC_Part_Number" "C7432791" (at 156.845 78.74 0)
       (effects (font (size 1.27 1.27)) hide)
     )
@@
       (effects (font (size 1.27 1.27)) hide)
     )
-    (property "Datasheet" "~" (at 123.825 69.215 0)
+    (property "Datasheet" "https://www.lcsc.com/product-detail/Multilayer-Ceramic-Capacitors-MLCC-SMD-SMT_CCTC-TCC0402X5R104K250AT_C880603.html" (at 123.825 69.215 0)
+      (effects (font (size 1.27 1.27)) hide)
+    )
+    (property "LCSC_Part_Number" "C880603" (at 123.825 69.215 0)
       (effects (font (size 1.27 1.27)) hide)
     )
@@
       (effects (font (size 1.27 1.27)) hide)
     )
-    (property "Datasheet" "~" (at 79.375 106.045 0)
+    (property "Datasheet" "https://www.lcsc.com/product-detail/Multilayer-Ceramic-Capacitors-MLCC-SMD-SMT_FH-Guangdong-Fenghua-Advanced-Tech-0201CG430J500NT_C3037638.html" (at 79.375 106.045 0)
+      (effects (font (size 1.27 1.27)) hide)
+    )
+    (property "LCSC_Part_Number" "C3037638" (at 79.375 106.045 0)
       (effects (font (size 1.27 1.27)) hide)
     )
@@
       (effects (font (size 1 1)) (justify bottom) hide)
     )
-    (property "Datasheet" "" (at 194.945 118.11 0)
+    (property "Datasheet" "https://www.lcsc.com/product-detail/USB-Connectors_SHOU-HAN-TYPE-C16P3MDDGP073_C2965608.html" (at 194.945 118.11 0)
       (effects (font (size 1.27 1.27)) hide)
     )
@@
       (effects (font (size 1.27 1.27)) (justify left top) hide)
     )
-    (property "Datasheet" "https://datasheet.lcsc.com/lcsc/2208111030_Samsung-Electro-Mechanics-CL10A226MO7JZNC_C2762594.pdf" (at 10.185 69.215 0)
+    (property "Datasheet" "https://www.lcsc.com/product-detail/Multilayer-Ceramic-Capacitors-MLCC-SMD-SMT_Samsung-Electro-Mechanics-CL10A226MO7JZNC_C2762594.html" (at 10.185 69.215 0)
       (effects (font (size 1.27 1.27)) (justify left top) hide)
     )
@@
       (effects (font (size 1.27 1.27)) hide)
     )
-    (property "Datasheet" "~" (at 93.98 143.51 0)
+    (property "Datasheet" "https://www.lcsc.com/product-detail/Multilayer-Ceramic-Capacitors-MLCC-SMD-SMT_Samsung-Electro-Mechanics-CL10A105KB8NNNC_C15849.html" (at 93.98 143.51 0)
+      (effects (font (size 1.27 1.27)) hide)
+    )
+    (property "LCSC_Part_Number" "C15849" (at 93.98 143.51 0)
       (effects (font (size 1.27 1.27)) hide)
     )
@@
       (effects (font (size 1.27 1.27)) hide)
     )
-    (property "Datasheet" "~" (at 55.245 79.375 0)
+    (property "Datasheet" "https://www.lcsc.com/product-detail/Multilayer-Ceramic-Capacitors-MLCC-SMD-SMT_HRE-CGA0603X5R475K250JT_C6119856.html" (at 55.245 79.375 0)
+      (effects (font (size 1.27 1.27)) hide)
+    )
+    (property "LCSC_Part_Number" "C6119856" (at 55.245 79.375 0)
       (effects (font (size 1.27 1.27)) hide)
     )
@@
       (effects (font (size 1.27 1.27)) hide)
     )
-    (property "Datasheet" "~" (at 43.815 79.375 0)
+    (property "Datasheet" "https://www.lcsc.com/product-detail/Multilayer-Ceramic-Capacitors-MLCC-SMD-SMT_CCTC-TCC0805X5R106K250FT_C5448891.html" (at 43.815 79.375 0)
+      (effects (font (size 1.27 1.27)) hide)
+    )
+    (property "LCSC_Part_Number" "C5448891" (at 43.815 79.375 0)
       (effects (font (size 1.27 1.27)) hide)
     )
@@
       (effects (font (size 1.27 1.27)) hide)
     )
-    (property "Datasheet" "~" (at 66.04 102.235 0)
-      (effects (font (size 1.27 1.27)) hide)
-    )
+    (property "Datasheet" "https://www.lcsc.com/product-detail/Multilayer-Ceramic-Capacitors-MLCC-SMD-SMT_FH-Guangdong-Fenghua-Advanced-Tech-0201X222K250NT_C285033.html" (at 66.04 102.235 0)
+      (effects (font (size 1.27 1.27)) hide)
+    )
+    (property "LCSC_Part_Number" "C285033" (at 66.04 102.235 0)
+      (effects (font (size 1.27 1.27)) hide)
+    )

Commit message: finished first pass on BOM. check 100uF cap and a couple others. TS
Parts:
- L1: LCSC_Part_Number (none) -> C2847540
- Q1: Field4 (none) -> pulled from excel sheet (TS) 5-31-24; LCSC_Part_Number (none) -> C5278892
- R16: LCSC_Part_Number (none) -> C2933066
- R17: LCSC_Part_Number (none) -> C25887
- R18: LCSC_Part_Number (none) -> C5153961
- R19: LCSC_Part_Number (none) -> C3013164
- R20: LCSC_Part_Number (none) -> C2906862
- R23: LCSC_Part_Number (none) -> C409700
- R24: LCSC_Part_Number (none) -> C2998086
- R25, R27: LCSC_Part_Number (none) -> C2906885
- R26: LCSC_Part_Number (none) -> C2906873
- R28: LCSC_Part_Number (none) -> C3015834
- R29: LCSC_Part_Number (none) -> C620467
- U6: LCSC_Part_Number (none) -> C263274
- U7: LCSC_Part_Number (none) -> C7471904
Changed lines of the file:
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@@
       (effects (font (size 1.27 1.27)) hide)
     )
-    (property "Datasheet" "~" (at 79.375 99.06 0)
+    (property "Datasheet" "https://www.lcsc.com/product-detail/Chip-Resistor-Surface-Mount_FOJAN-FRC0402F3401TS_C3013164.html" (at 79.375 99.06 0)
+      (effects (font (size 1.27 1.27)) hide)
+    )
+    (property "LCSC_Part_Number" "C3013164" (at 79.375 99.06 0)
       (effects (font (size 1.27 1.27)) hide)
     )
@@
       (effects (font (size 1.27 1.27)) hide)
     )
-    (property "Datasheet" "" (at 120.015 145.9738 0)
+    (property "Datasheet" "https://www.lcsc.com/product-detail/span-style-background-color-ff0-USB-span-Converters_Hynetek-HUSB238_002DD_C7471904.html" (at 120.015 145.9738 0)
       (effects (font (size 1.27 1.27)) hide)
     )
@@
     )
     (property "uuid" "std:72c35b3c087241289ee1276473b7df23" (at 120.015 151.0538 0)
+      (effects (font (size 1.27 1.27)) hide)
+    )
+    (property "LCSC_Part_Number" "C7471904" (at 120.015 146.05 0)
       (effects (font (size 1.27 1.27)) hide)
     )
@@
       (effects (font (size 1.27 1.27)) hide)
     )
-    (property "Datasheet" "~" (at 104.775 135.89 0)
+    (property "Datasheet" "https://www.lcsc.com/product-detail/Chip-Resistor-Surface-Mount_FOJAN-FRC0402F10R0TS_C2906862.html" (at 104.775 135.89 0)
+      (effects (font (size 1.27 1.27)) hide)
+    )
+    (property "LCSC_Part_Number" "C2906862" (at 104.775 135.89 0)
       (effects (font (size 1.27 1.27)) hide)
     )
@@
       (effects (font (size 1.27 1.27)) hide)
     )
-    (property "Datasheet" "~" (at 152.4 133.985 0)
+    (property "Datasheet" "https://www.lcsc.com/product-detail/MOSFETs_PAKER-SI2323_C5278892.html" (at 152.4 133.985 0)
+      (effects (font (size 1.27 1.27)) hide)
+    )
+    (property "Field4" "pulled from excel sheet (TS) 5-31-24" (at 152.4 133.985 0)
+      (effects (font (size 1.27 1.27)) hide)
+    )
+    (property "LCSC_Part_Number" "C5278892" (at 152.4 133.985 0)
       (effects (font (size 1.27 1.27)) hide)
     )
@@
       (effects (font (size 1.27 1.27)) hide)
     )
-    (property "Datasheet" "~" (at 138.43 140.97 0)
+    (property "Datasheet" "https://www.lcsc.com/product-detail/Chip-Resistor-Surface-Mount_Viking-Tech-CR-02FL6-5K1_C409700.html" (at 138.43 140.97 0)
+      (effects (font (size 1.27 1.27)) hide)
+    )
+    (property "LCSC_Part_Number" "C409700" (at 138.43 140.97 0)
       (effects (font (size 1.27 1.27)) hide)
     )
@@
       (effects (font (size 1.27 1.27)) hide)
     )
-    (property "Datasheet" "~" (at 73.66 99.06 0)
+    (property "Datasheet" "https://www.lcsc.com/product-detail/Chip-Resistor-Surface-Mount_FOJAN-FRC0402F5362TS_C5153961.html" (at 73.66 99.06 0)
+      (effects (font (size 1.27 1.27)) hide)
+    )
+    (property "LCSC_Part_Number" "C5153961" (at 73.66 99.06 0)
       (effects (font (size 1.27 1.27)) hide)
     )
@@
       (effects (font (size 1.27 1.27)) hide)
     )
-    (property "Datasheet" "~" (at 142.875 71.755 0)
+    (property "Datasheet" "https://www.lcsc.com/product-detail/Chip-Resistor-Surface-Mount_FOJAN-FRC0402F5232TS_C2998086.html" (at 142.875 71.755 0)
+      (effects (font (size 1.27 1.27)) hide)
+    )
+    (property "LCSC_Part_Number" "C2998086" (at 142.875 71.755 0)
       (effects (font (size 1.27 1.27)) hide)
     )
@@
       (effects (font (size 1.27 1.27)) hide)
     )
-    (property "Datasheet" "~" (at 146.685 169.545 0)
+    (property "Datasheet" "https://www.lcsc.com/product-detail/Chip-Resistor-Surface-Mount_FOJAN-FRC0402J103-TS_C2906885.html" (at 146.685 169.545 0)
+      (effects (font (size 1.27 1.27)) hide)
+    )
+    (property "LCSC_Part_Number" "C2906885" (at 146.685 169.545 0)
       (effects (font (size 1.27 1.27)) hide)
     )
@@
       (effects (font (size 1.27 1.27)) hide)
     )
-    (property "Datasheet" "~" (at 60.96 86.36 0)
+    (property "Datasheet" "https://www.lcsc.com/product-detail/Chip-Resistor-Surface-Mount_UNI-ROYAL-Uniroyal-Elec-0402WGF3652TCE_C25887.html" (at 60.96 86.36 0)
+      (effects (font (size 1.27 1.27)) hide)
+    )
+    (property "LCSC_Part_Number" "C25887" (at 60.96 86.36 0)
       (effects (font (size 1.27 1.27)) hide)
     )
@@
       (effects (font (size 1.27 1.27)) hide)
     )
-    (property "Datasheet" "~" (at 134.62 65.405 0)
+    (property "Datasheet" "https://www.lcsc.com/product-detail/Inductors-SMD_KOHERelec-MDA7050-3R3M_C2847540.html" (at 134.62 65.405 0)
+      (effects (font (size 1.27 1.27)) hide)
+    )
+    (property "LCSC_Part_Number" "C2847540" (at 134.62 65.405 0)
       (effects (font (size 1.27 1.27)) hide)
     )
@@
       (effects (font (size 1.27 1.27)) hide)
     )
-    (property "Datasheet" "~" (at 145.415 136.525 0)
+    (property "Datasheet" "https://www.lcsc.com/product-detail/Chip-Resistor-Surface-Mount_FOJAN-FRC0402F4992TS_C2906873.html" (at 145.415 136.525 0)
+      (effects (font (size 1.27 1.27)) hide)
+    )
+    (property "LCSC_Part_Number" "C2906873" (at 145.415 136.525 0)
       (effects (font (size 1.27 1.27)) hide)
     )
@@
       (effects (font (size 1.27 1.27)) hide)
     )
-    (property "Datasheet" "http://www.szlcsc.com/product/details_254511.html" (at 97.79 70.4088 0)
+    (property "Datasheet" "https://www.lcsc.com/product-detail/DC-DC-Converters_Texas-Instruments-TPS54620RHLR_C263274.html" (at 97.79 70.4088 0)
       (effects (font (size 1.27 1.27)) hide)
     )
@@
     )
     (property "uuid" "std:22c093bd3f0e4f169efe6636adc161b3" (at 97.79 75.4888 0)
+      (effects (font (size 1.27 1.27)) hide)
+    )
+    (property "LCSC_Part_Number" "C263274" (at 97.79 80.645 0)
       (effects (font (size 1.27 1.27)) hide)
     )
@@
       (effects (font (size 1.27 1.27)) hide)
     )
-    (property "Datasheet" "~" (at 159.385 168.91 0)
+    (property "Datasheet" "https://www.lcsc.com/product-detail/Chip-Resistor-Surface-Mount_UNI-ROYAL-Uniroyal-Elec-0402WGF105JTCE_C620467.html" (at 159.385 168.91 0)
+      (effects (font (size 1.27 1.27)) hide)
+    )
+    (property "LCSC_Part_Number" "C620467" (at 159.385 168.91 0)
       (effects (font (size 1.27 1.27)) hide)
     )
@@
       (effects (font (size 1.27 1.27)) hide)
     )
-    (property "Datasheet" "~" (at 142.875 87.63 0)
+    (property "Datasheet" "https://www.lcsc.com/product-detail/Chip-Resistor-Surface-Mount_FOJAN-FRC0402J103-TS_C2906885.html" (at 142.875 87.63 0)
+      (effects (font (size 1.27 1.27)) hide)
+    )
+    (property "LCSC_Part_Number" "C2906885" (at 142.875 87.63 0)
       (effects (font (size 1.27 1.27)) hide)
     )
@@
       (effects (font (size 1.27 1.27)) hide)
     )
-    (property "Datasheet" "http://www.advanced-monolithic.com/pdf/ds1117.pdf" (at 198.12 65.405 0)
+    (property "Datasheet" "https://www.lcsc.com/product-detail/Linear-Voltage-Regulators-LDO_UMW-Youtai-Semiconductor-Co-Ltd-AMS1117-3-3_C347222.html" (at 198.12 65.405 0)
       (effects (font (size 1.27 1.27)) hide)
     )
@@
       (effects (font (size 1.27 1.27)) hide)
     )
-    (property "Datasheet" "~" (at 60.96 75.565 0)
+    (property "Datasheet" "https://www.lcsc.com/product-detail/Chip-Resistor-Surface-Mount_FOJAN-FRC0402F1023TS_C2933066.html" (at 60.96 75.565 0)
+      (effects (font (size 1.27 1.27)) hide)
+    )
+    (property "LCSC_Part_Number" "C2933066" (at 60.96 75.565 0)
       (effects (font (size 1.27 1.27)) hide)
     )
@@
       (effects (font (size 1.27 1.27)) hide)
     )
-    (property "Datasheet" "~" (at 150.495 169.545 0)
-      (effects (font (size 1.27 1.27)) hide)
-    )
+    (property "Datasheet" "https://www.lcsc.com/product-detail/Chip-Resistor-Surface-Mount_VO-SCR0402F14K_C3015834.html" (at 150.495 169.545 0)
+      (effects (font (size 1.27 1.27)) hide)
+    )
+    (property "LCSC_Part_Number" "C3015834" (at 150.495 169.545 0)
+      (effects (font (size 1.27 1.27)) hide)
+    )
