File: motorgo_plink/motorgo_plink.kicad_sch (KiCad schematic)
At the start: 23 parts, among them J1 USB4520-03-0-A_REVA, J4 Conn_02x20_Odd_Even, U1 ESP32-S3-WROOM-1, U2 USBLC6-2P6

Commit message: replaced female 2x20 header with brick nogging. male pin headers listed in the google sheets.
Parts:
- J4: LCSC_Part_Number C2977589 -> C3975165
Changed lines of the file:
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@@
       (effects (font (size 1.27 1.27)) hide)
     )
-    (property "Datasheet" "https://www.lcsc.com/product-detail/Female-Headers_ZHOURI-2-54-2-20_C2977589.html" (at 230.505 45.72 0)
+    (property "Datasheet" "https://www.lcsc.com/product-detail/Female-Headers_HCTL-PM254-2-20-S-8-5_C3975165.html" (at 230.505 45.72 0)
       (effects (font (size 1.27 1.27)) hide)
     )
@@
       (effects (font (size 1.27 1.27)) hide)
     )
-    (property "LCSC_Part_Number" "C2977589" (at 230.505 45.72 0)
+    (property "LCSC_Part_Number" "C3975165" (at 230.505 45.72 0)
       (effects (font (size 1.27 1.27)) hide)
     )
