File: motorgo_plink/motorgo_plink.kicad_sch (KiCad schematic)
At the start: 24 parts, among them J11 USB4520-03-0-A_REVA, J21 Conn_02x20_Odd_Even, J8 Conn_02x20_Odd_Even, U1 ESP32-S3-WROOM-1, U8 USBLC6-2P6

Commit message: WIP update, schematic mainly complete
Other:
- sheet IMU 6 + 3 ports: added SCL, SDA; removed none
- sheet Power Reg and Dist ports: added scl_pd, sda_pd; removed none
Changed lines of the file:
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@@
       (effects (font (size 1.27 1.27)) (justify left top))
+    )
+    (pin "SCL" input (at 157.48 133.35 180)
+      (effects (font (size 1.27 1.27)) (justify left))
+    )
+    (pin "SDA" input (at 157.48 135.89 180)
+      (effects (font (size 1.27 1.27)) (justify left))
     )
     (instances
@@
       (effects (font (size 1.27 1.27)) hide)
     )
+    (pin "scl_pd" input (at 158.115 97.79 180)
+      (effects (font (size 1.27 1.27)) (justify left))
+    )
+    (pin "sda_pd" input (at 158.115 100.33 180)
+      (effects (font (size 1.27 1.27)) (justify left))
+    )
     (instances

Commit message: WIP update. Parts semi-finalized
Parts:
- removed J8: Conn_02x20_Odd_Even, symbol Connector_Generic:Conn_02x20_Odd_Even
- J1: renamed from J11; footprint aaa_motorgo_components:GCT_USB4520-03-0-A_REVA -> mg_mini_v1r3:GCT_USB4520-03-0-A_REVA
- J4: renamed from J21; footprint (none) -> Connector_PinHeader_2.54mm:PinHeader_2x20_P2.54mm_Vertical_SMD
- U1: footprint aaa_espressif_github:ESP32-S3-WROOM-1 -> mg_mini_v1r3:ESP32-S3-WROOM-1
- renumbered J7 to J2, J6 to J3, R32 to R1, R22 to R2, R33 to R3, R23 to R4, R24 to R5, R21 to R6, R20 to R7, R25 to R8, R30 to R9, U8 to U2
Connections:
- net gpio6 is gone; now on net gpio4: J4.12 (Pin_12)
- net p21 is gone; now on net gpio39: J4.21 (Pin_21)
- net p22 is gone; now on net gpio41: J4.22 (Pin_22)
- net p23 is gone; now on net gpio40: J4.23 (Pin_23)
- net p24 is gone; now on net gpio42: J4.24 (Pin_24)
- net p25 is gone; now on net GND: J4.25 (Pin_25)
- net p30 is gone; now on net GND: J4.30 (Pin_30)
- net p34 is gone; now on net GND: J4.34 (Pin_34)
- net p39 is gone; now on net GND: J4.39 (Pin_39)
- net gpio7: now also U1.7 (GPIO7/TOUCH7/ADC1_CH6)
- net gpio8: now also U1.12 (GPIO8/TOUCH8/ADC1_CH7/SUBSPICS1)
- net gpio9: now also U1.17 (GPIO9/TOUCH9/ADC1_CH8/FSPIHD/SUBSPIHD)
- net hidden_scl: now reaches U1.5 (GPIO5/TOUCH5/ADC1_CH4)
- net hidden_sda: now reaches U1.6 (GPIO6/TOUCH6/ADC1_CH5)
- net m1_vl renamed m4_enc_cs
- net m1_wl renamed m3_enc_cs
- net p27: no longer names the net of J4.27 (Pin_27)
- net p28: no longer names the net of J4.28 (Pin_28)
- no-connect marks 8 -> 10
Other:
- note added: "Pass through pins"
- note added: "The ADC2 Channels do not perform as expected with the wifi capabilities of the ESP32"
- moved on the sheet: J4

Commit message: WIP update. Layout begin
Connections:
- net p29 is gone; now on net boot: J4.29 (Pin_29)
- net gpio38: now also J4.24 (Pin_24); no longer J4.19 (Pin_19)
- net gpio42: now also J4.19 (Pin_19); no longer J4.24 (Pin_24)
Changed lines of the file:
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@@
+    (stroke (width 0) (type default))
+  )
+  (wire (pts (xy 213.995 40.64) (xy 225.425 40.64))
     (stroke (width 0) (type default))
   )
@@
   )
   (polyline (pts (xy 217.805 109.855) (xy 217.17 109.22))
+    (stroke (width 0) (type default))
+  )
+  (wire (pts (xy 213.36 58.42) (xy 225.425 58.42))
     (stroke (width 0) (type default))
   )
@@
     )
   )
-  (global_label "gpio42" (shape input) (at 238.125 50.8 0) (fields_autoplaced)
-    (effects (font (size 1.27 1.27)) (justify left))
-    (property "Intersheetrefs" "${INTERSHEET_REFS}" (at 247.5016 50.8 0)
-      (effects (font (size 1.27 1.27)) (justify left) hide)
+  (global_label "gpio42" (shape input) (at 225.425 45.72 180) (fields_autoplaced)
+    (effects (font (size 1.27 1.27)) (justify right))
+    (property "Intersheetrefs" "${INTERSHEET_REFS}" (at 216.0484 45.72 0)
+      (effects (font (size 1.27 1.27)) (justify right) hide)
     )
   )
@@
     )
   )
+  (global_label "boot" (shape input) (at 213.36 58.42 180) (fields_autoplaced)
+    (effects (font (size 1.27 1.27)) (justify right))
+    (property "Intersheetrefs" "${INTERSHEET_REFS}" (at 206.2815 58.42 0)
+      (effects (font (size 1.27 1.27)) (justify right) hide)
+    )
+  )
   (global_label "m2_PH" (shape input) (at 226.06 112.395 180) (fields_autoplaced)
     (effects (font (size 1.27 1.27) (color 255 255 0 1)) (justify right))
@@
     )
   )
-  (global_label "Reset" (shape input) (at 225.425 40.64 180) (fields_autoplaced)
-    (effects (font (size 1.27 1.27)) (justify right))
-    (property "Intersheetrefs" "${INTERSHEET_REFS}" (at 217.3182 40.64 0)
+  (global_label "Reset" (shape input) (at 213.995 40.64 180) (fields_autoplaced)
+    (effects (font (size 1.27 1.27)) (justify right))
+    (property "Intersheetrefs" "${INTERSHEET_REFS}" (at 205.8882 40.64 0)
       (effects (font (size 1.27 1.27)) (justify right) hide)
     )
@@
     )
   )
-  (global_label "gpio38" (shape input) (at 225.425 45.72 180) (fields_autoplaced)
-    (effects (font (size 1.27 1.27)) (justify right))
-    (property "Intersheetrefs" "${INTERSHEET_REFS}" (at 216.0484 45.72 0)
-      (effects (font (size 1.27 1.27)) (justify right) hide)
+  (global_label "gpio38" (shape input) (at 238.125 50.8 0) (fields_autoplaced)
+    (effects (font (size 1.27 1.27)) (justify left))
+    (property "Intersheetrefs" "${INTERSHEET_REFS}" (at 247.5016 50.8 0)
+      (effects (font (size 1.27 1.27)) (justify left) hide)
     )
   )
@@
     )
   )
-  (global_label "p29" (shape input) (at 225.425 58.42 180) (fields_autoplaced)
-    (effects (font (size 1.27 1.27)) (justify right))
-    (property "Intersheetrefs" "${INTERSHEET_REFS}" (at 218.9512 58.42 0)
-      (effects (font (size 1.27 1.27)) (justify right) hide)
-    )
-  )

Commit message: WIP update. Ready for BOM editing
Parts:
- J4: footprint Connector_PinHeader_2.54mm:PinHeader_2x20_P2.54mm_Vertical_SMD -> Connector_PinSocket_2.54mm:PinSocket_2x20_P2.54mm_Vertical_SMD
Other:
- note added: "GPIO link to Rpi"
- note removed: "GPIO link to Rpi (top and bottom side)"
- moved on the sheet: C2, J1, R4, R5, R6, R7, U2

Commit message: WIP update. change USBC port
Parts:
- J1: footprint mg_mini_v1r3:GCT_USB4520-03-0-A_REVA -> mg_mini_v1r3:USB-C-SMD_TYPEC-303-ACP16
Connections:
- net +5V: now also J1.A4 (Vbus), J1.A9 (VBUS), J1.B4 (VBUS), J1.B9 (VBUS); no longer J1.A4_B9 (VBUS_A), J1.B4_A9 (VBUS_B)
- net GND: now also J1.1 (SHELL_GND), J1.2 (SHELL_GND), J1.3 (SHELL_GND), J1.4 (SHELL_GND), J1.A1 (GND), J1.A12 (GND), J1.B1 (GND), J1.B12 (GND); no longer J1.A1_B12 (GND_A), J1.B1_A12 (GND_B)
- net enc_scl: now also U1.7 (GPIO7/TOUCH7/ADC1_CH6); no longer U1.29 (SPIIO7/GPIO36/FSPICLK/SUBSPICLK)
- net enc_sda: now also U1.6 (GPIO6/TOUCH6/ADC1_CH5); no longer U1.28 (SPIIO6/GPIO35/FSPID/SUBSPID)
- net gpio3: now also U1.30 (SPIDQS/GPIO37/FSPIQ/SUBSPIQ); no longer U1.15 (GPIO3/TOUCH3/ADC1_CH2)
- net gpio38: now also U1.23 (GPIO21); no longer U1.31 (GPIO38/FSPIWP/SUBSPIWP)
- net gpio4: now also U1.28 (SPIIO6/GPIO35/FSPID/SUBSPID); no longer U1.4 (GPIO4/TOUCH4/ADC1_CH3)
- net gpio41: now also U1.24 (GPIO47/SPICLK_P/SUBSPICLK_P_DIFF); no longer U1.34 (MTDI/GPIO41/CLK_OUT1)
- net gpio42: now also U1.25 (GPIO48/SPICLK_N/SUBSPICLK_N_DIFF); no longer U1.35 (MTMS/GPIO42)
- net gpio43: now also J4.8 (Pin_8), U1.36 (U0RXD/GPIO44/CLK_OUT2); no longer J4.10 (Pin_10), U1.37 (U0TXD/GPIO43/CLK_OUT1)
- net gpio44: now also J4.10 (Pin_10), U1.34 (MTDI/GPIO41/CLK_OUT1); no longer J4.8 (Pin_8), U1.36 (U0RXD/GPIO44/CLK_OUT2)
- net gpio47: now also U1.35 (MTMS/GPIO42); no longer U1.24 (GPIO47/SPICLK_P/SUBSPICLK_P_DIFF)
- net gpio7: now also U1.29 (SPIIO7/GPIO36/FSPICLK/SUBSPICLK); no longer U1.7 (GPIO7/TOUCH7/ADC1_CH6)
- net gpio8: now also U1.31 (GPIO38/FSPIWP/SUBSPIWP); no longer U1.12 (GPIO8/TOUCH8/ADC1_CH7/SUBSPICS1)
- net gpio9: now also U1.37 (U0TXD/GPIO43/CLK_OUT1); no longer U1.17 (GPIO9/TOUCH9/ADC1_CH8/FSPIHD/SUBSPIHD)
- net hidden_scl: now also U1.22 (GPIO14/TOUCH14/ADC2_CH3/FSPIWP/FSPIDQS/SUBSPIWP); no longer U1.5 (GPIO5/TOUCH5/ADC1_CH4)
- net hidden_sda: now also U1.21 (GPIO13/TOUCH13/ADC2_CH2/FSPIQ/FSPIIO7/SUBSPIQ); no longer U1.6 (GPIO6/TOUCH6/ADC1_CH5)
- net m1_EN: now also U1.9 (GPIO16/U0CTS/ADC2_CH5/XTAL_32K_N); no longer U1.18 (GPIO10/TOUCH10/ADC1_CH9/FSPICS0/FSPIIO4/SUBSPICS0)
- net m1_PH: now also U1.8 (GPIO15/U0RTS/ADC2_CH4/XTAL_32K_P); no longer U1.19 (GPIO11/TOUCH11/ADC2_CH0/FSPID/FSPIIO5/SUBSPID)
- net m1_enc_cs: now also U1.5 (GPIO5/TOUCH5/ADC1_CH4); no longer U1.30 (SPIDQS/GPIO37/FSPIQ/SUBSPIQ)
- net m2_EN: now also U1.11 (GPIO18/U1RXD/ADC2_CH7/CLK_OUT3); no longer U1.20 (GPIO12/TOUCH12/ADC2_CH1/FSPICLK/FSPIIO6/SUBSPICLK)
- net m2_PH: now also U1.10 (GPIO17/U1TXD/ADC2_CH6); no longer U1.21 (GPIO13/TOUCH13/ADC2_CH2/FSPIQ/FSPIIO7/SUBSPIQ)
- net m2_enc_cs: now also U1.4 (GPIO4/TOUCH4/ADC1_CH3); no longer U1.25 (GPIO48/SPICLK_N/SUBSPICLK_N_DIFF)
- net m3_EN: now also U1.15 (GPIO3/TOUCH3/ADC1_CH2); no longer U1.22 (GPIO14/TOUCH14/ADC2_CH3/FSPIWP/FSPIDQS/SUBSPIWP)
- net m3_PH: now also U1.12 (GPIO8/TOUCH8/ADC1_CH7/SUBSPICS1); no longer U1.10 (GPIO17/U1TXD/ADC2_CH6)
- net m3_enc_cs: now also U1.17 (GPIO9/TOUCH9/ADC1_CH8/FSPIHD/SUBSPIHD); no longer U1.8 (GPIO15/U0RTS/ADC2_CH4/XTAL_32K_P)
- net m4_EN: now also U1.19 (GPIO11/TOUCH11/ADC2_CH0/FSPID/FSPIIO5/SUBSPID); no longer U1.11 (GPIO18/U1RXD/ADC2_CH7/CLK_OUT3)
- net m4_PH: now also U1.18 (GPIO10/TOUCH10/ADC1_CH9/FSPICS0/FSPIIO4/SUBSPICS0); no longer U1.23 (GPIO21)
- net m4_enc_cs: now also U1.20 (GPIO12/TOUCH12/ADC2_CH1/FSPICLK/FSPIIO6/SUBSPICLK); no longer U1.9 (GPIO16/U0CTS/ADC2_CH5/XTAL_32K_N)
- no-connect marks 10 -> 6

Commit message: ready for order
Parts:
- removed C2 (x2): DNP, Capacitor_SMD:C_0402_1005Metric, symbol sparkfun_capacitors:0.1UF-0402-16V-10%
Changed lines of the file:
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@@
   (junction (at 132.715 155.575) (diameter 0) (color 0 0 0 0)
-  )
-  (junction (at 132.715 180.34) (diameter 0) (color 0 0 0 0)
   )
   (junction (at 120.015 145.415) (diameter 0) (color 0 0 0 0)
@@
     (stroke (width 0) (type default))
   )
-  (wire (pts (xy 132.715 186.69) (xy 132.715 187.96))
-    (stroke (width 0) (type default))
-  )
   (wire (pts (xy 113.03 155.575) (xy 113.03 158.75))
     (stroke (width 0) (type default))
@@
     (stroke (width 0) (type default))
   )
-  (wire (pts (xy 132.715 162.56) (xy 132.715 163.83))
-    (stroke (width 0) (type default))
-  )
   (wire (pts (xy 118.11 155.575) (xy 118.11 158.75))
     (stroke (width 0) (type default))
   )
-  (wire (pts (xy 132.715 180.34) (xy 131.445 180.34))
-    (stroke (width 0) (type default))
-  )
   (wire (pts (xy 238.125 22.86) (xy 238.125 25.4))
     (stroke (width 0) (type default))
@@
     (stroke (width 0) (type default))
   )
-  (wire (pts (xy 133.985 180.34) (xy 132.715 180.34))
+  (wire (pts (xy 131.445 180.34) (xy 133.985 180.34))
     (stroke (width 0) (type default))
   )
@@
         (path "/e63e39d7-6ac0-4ffd-8aa3-1841a4541b55/c5a81061-28ff-4599-a380-43adb8d460db"
           (reference "#PWR030") (unit 1)
-        )
-      )
-    )
-  )
-  (symbol (lib_id "sparkfun_capacitors:0.1UF-0402-16V-10%") (at 132.715 182.88 180) (unit 1)
-    (in_bom yes) (on_board yes) (dnp no)
-    (property "Reference" "C2" (at 134.62 186.055 0)
-      (effects (font (size 1.143 1.143)))
-    )
-    (property "Value" "DNP" (at 139.065 184.15 0)
-      (effects (font (size 1.143 1.143)))
-    )
-    (property "Footprint" "Capacitor_SMD:C_0402_1005Metric" (at 132.715 189.23 0)
-      (effects (font (size 0.508 0.508)) hide)
-    )
-    (property "Datasheet" "" (at 132.715 182.88 0)
-      (effects (font (size 1.27 1.27)) hide)
-    )
-    (property "Field4" "CAP-12416" (at 128.905 184.15 90)
-      (effects (font (size 1.524 1.524)) hide)
-    )
-    (property "LCSC_Part_Number" "-" (at 132.715 182.88 0)
-      (effects (font (size 1.27 1.27)) hide)
-    )
-    (pin "1")
-    (pin "2")
-    (instances
-      (project "motorgo_plink"
-        (path "/e63e39d7-6ac0-4ffd-8aa3-1841a4541b55/47ec5f88-3723-4b64-bf75-8726c250fd67"
-          (reference "C2") (unit 1)
-        )
-        (path "/e63e39d7-6ac0-4ffd-8aa3-1841a4541b55"
-          (reference "C2") (unit 1)
         )
       )
@@
     )
   )
-  (symbol (lib_id "power:GND") (at 132.715 186.69 0) (unit 1)
-    (in_bom yes) (on_board yes) (dnp no) (fields_autoplaced)
-    (property "Reference" "#PWR013" (at 132.715 193.04 0)
-      (effects (font (size 1.27 1.27)) hide)
-    )
-    (property "Value" "GND" (at 132.715 191.77 0)
-      (effects (font (size 1.27 1.27)))
-    )
-    (property "Footprint" "" (at 132.715 186.69 0)
-      (effects (font (size 1.27 1.27)) hide)
-    )
-    (property "Datasheet" "" (at 132.715 186.69 0)
-      (effects (font (size 1.27 1.27)) hide)
-    )
-    (pin "1")
-    (instances
-      (project "motorgo_plink"
-        (path "/e63e39d7-6ac0-4ffd-8aa3-1841a4541b55"
-          (reference "#PWR013") (unit 1)
-        )
-      )
-    )
-  )
   (symbol (lib_id "Graphic:Logo_Open_Hardware_Small") (at 166.37 179.07 0) (unit 1)
     (in_bom no) (on_board no) (dnp no) (fields_autoplaced)
@@
         )
       )
-    )
-  )
-  (symbol (lib_id "sparkfun_capacitors:0.1UF-0402-16V-10%") (at 132.715 158.75 180) (unit 1)
-    (in_bom yes) (on_board yes) (dnp no)
-    (property "Reference" "C2" (at 134.62 161.925 0)
-      (effects (font (size 1.143 1.143)))
-    )
-    (property "Value" "DNP" (at 139.065 160.02 0)
-      (effects (font (size 1.143 1.143)))
-    )
-    (property "Footprint" "Capacitor_SMD:C_0402_1005Metric" (at 132.715 165.1 0)
-      (effects (font (size 0.508 0.508)) hide)
-    )
-    (property "Datasheet" "" (at 132.715 158.75 0)
-      (effects (font (size 1.27 1.27)) hide)
-    )
-    (property "Field4" "CAP-12416" (at 128.905 160.02 90)
-      (effects (font (size 1.524 1.524)) hide)
-    )
-    (property "LCSC_Part_Number" "-" (at 132.715 158.75 0)
-      (effects (font (size 1.27 1.27)) hide)
-    )
-    (pin "1")
-    (pin "2")
-    (instances
-      (project "motorgo_plink"
-        (path "/e63e39d7-6ac0-4ffd-8aa3-1841a4541b55/47ec5f88-3723-4b64-bf75-8726c250fd67"
-          (reference "C2") (unit 1)
-        )
-        (path "/e63e39d7-6ac0-4ffd-8aa3-1841a4541b55"
-          (reference "C1") (unit 1)
-        )
-      )
-    )
-  )
-  (symbol (lib_id "power:GND") (at 132.715 162.56 0) (unit 1)
-    (in_bom yes) (on_board yes) (dnp no) (fields_autoplaced)
-    (property "Reference" "#PWR012" (at 132.715 168.91 0)
-      (effects (font (size 1.27 1.27)) hide)
-    )
-    (property "Value" "GND" (at 132.715 167.64 0)
-      (effects (font (size 1.27 1.27)))
-    )
-    (property "Footprint" "" (at 132.715 162.56 0)
-      (effects (font (size 1.27 1.27)) hide)
-    )
-    (property "Datasheet" "" (at 132.715 162.56 0)
-      (effects (font (size 1.27 1.27)) hide)
-    )
-    (pin "1")
-    (instances
-      (project "motorgo_plink"
-        (path "/e63e39d7-6ac0-4ffd-8aa3-1841a4541b55"
-          (reference "#PWR012") (unit 1)
-        )
-      )

Commit message: updated BOM in prep for order - TS
Parts:
- J1: LCSC_Part_Number C2965608 -> C720628
- J4: LCSC_Part_Number (none) -> C3975165
- R1, R2, R3: LCSC_Part_Number C100195 -> C2906899
- R6, R7: LCSC_Part_Number C163812 -> C3017451
Changed lines of the file:
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@@
       (effects (font (size 0.508 0.508)) hide)
     )
-    (property "Datasheet" "" (at 114.935 147.955 0)
+    (property "Datasheet" "https://www.lcsc.com/product-detail/Chip-Resistor-Surface-Mount_Viking-Tech-CR-02FL6-5K1_C409700.html" (at 114.935 147.955 0)
       (effects (font (size 1.524 1.524)) hide)
     )
@@
       (effects (font (size 0.508 0.508)) hide)
     )
-    (property "Datasheet" "" (at 167.64 29.21 0)
+    (property "Datasheet" "https://www.lcsc.com/product-detail/Chip-Resistor-Surface-Mount_Viking-Tech-CR-02FL6-5K1_C409700.html" (at 167.64 29.21 0)
       (effects (font (size 1.524 1.524)) hide)
     )
@@
       (effects (font (size 0.508 0.508)) hide)
     )
-    (property "Datasheet" "" (at 183.515 29.21 0)
+    (property "Datasheet" "https://www.lcsc.com/product-detail/Chip-Resistor-Surface-Mount_Viking-Tech-CR-02FL6-5K1_C409700.html" (at 183.515 29.21 0)
       (effects (font (size 1.524 1.524)) hide)
     )
@@
       (effects (font (size 0.508 0.508)) hide)
     )
-    (property "Datasheet" "" (at 25.4 174.625 0)
+    (property "Datasheet" "https://www.lcsc.com/product-detail/Chip-Resistor-Surface-Mount_FOJAN-FRC0402J102-TS_C2906899.html" (at 25.4 174.625 0)
       (effects (font (size 1.524 1.524)) hide)
     )
@@
       (effects (font (size 1.524 1.524)) (justify right))
     )
-    (property "LCSC_Part_Number" "C100195" (at 25.4 174.625 0)
+    (property "LCSC_Part_Number" "C2906899" (at 25.4 174.625 0)
       (effects (font (size 1.27 1.27)) hide)
     )
@@
       (effects (font (size 1.27 1.27)) hide)
     )
-    (property "Datasheet" "https://www.espressif.com/sites/default/files/documentation/esp32-s3-wroom-1_wroom-1u_datasheet_en.pdf" (at 85.725 116.84 0)
+    (property "Datasheet" "https://www.lcsc.com/product-detail/WiFi-Modules_Espressif-Systems-ESP32-S3-WROOM-1-N8_C2913198.html" (at 85.725 116.84 0)
       (effects (font (size 1.27 1.27)) hide)
     )
@@
       (effects (font (size 0.508 0.508)) hide)
     )
-    (property "Datasheet" "" (at 44.45 174.625 0)
+    (property "Datasheet" "https://www.lcsc.com/product-detail/Chip-Resistor-Surface-Mount_FOJAN-FRC0402J102-TS_C2906899.html" (at 44.45 174.625 0)
       (effects (font (size 1.524 1.524)) hide)
     )
@@
       (effects (font (size 1.524 1.524)) (justify right))
     )
-    (property "LCSC_Part_Number" "C100195" (at 44.45 174.625 0)
+    (property "LCSC_Part_Number" "C2906899" (at 44.45 174.625 0)
       (effects (font (size 1.27 1.27)) hide)
     )
@@
       (effects (font (size 1.27 1.27)) hide)
     )
-    (property "Datasheet" "https://www.st.com/resource/en/datasheet/usblc6-2.pdf" (at 124.46 173.99 0)
+    (property "Datasheet" "https://www.lcsc.com/product-detail/Electrostatic-and-Surge-Protection-TVS-ESD_TECH-PUBLIC-USBLC6-2P6_C2827693.html" (at 124.46 173.99 0)
       (effects (font (size 1.27 1.27)) hide)
     )
@@
       (effects (font (size 1 1)) (justify bottom) hide)
     )
-    (property "Datasheet" "" (at 73.025 154.305 0)
+    (property "Datasheet" "https://www.lcsc.com/product-detail/USB-Connectors_XUNPU-TYPEC-303-ACP16_C720628.html" (at 73.025 154.305 0)
       (effects (font (size 1.27 1.27)) hide)
     )
@@
       (effects (font (size 1.27 1.27)) (justify bottom) hide)
     )
-    (property "LCSC_Part_Number" "C2965608" (at 73.025 154.305 0)
+    (property "LCSC_Part_Number" "C720628" (at 73.025 154.305 0)
       (effects (font (size 1.27 1.27)) hide)
     )
@@
       (effects (font (size 1.27 1.27)) hide)
     )
-    (property "Datasheet" "~" (at 172.72 40.005 0)
+    (property "Datasheet" "https://www.lcsc.com/product-detail/Tactile-Switches_E-Switch-TL3342F450QG_C2886897.html" (at 172.72 40.005 0)
       (effects (font (size 1.27 1.27)) hide)
     )
@@
       (effects (font (size 0.508 0.508)) hide)
     )
-    (property "Datasheet" "" (at 114.935 145.415 0)
+    (property "Datasheet" "https://www.lcsc.com/product-detail/Chip-Resistor-Surface-Mount_Viking-Tech-CR-02FL6-5K1_C409700.html" (at 114.935 145.415 0)
       (effects (font (size 1.524 1.524)) hide)
     )
@@
       (effects (font (size 1.27 1.27)) hide)
     )
-    (property "Datasheet" "~" (at 230.505 45.72 0)
+    (property "Datasheet" "https://www.lcsc.com/product-detail/Female-Headers_HCTL-PM254-2-20-S-8-5_C3975165.html" (at 230.505 45.72 0)
+      (effects (font (size 1.27 1.27)) hide)
+    )
+    (property "LCSC_Part_Number" "C3975165" (at 230.505 45.72 0)
       (effects (font (size 1.27 1.27)) hide)
     )
@@
       (effects (font (size 1.27 1.27)) hide)
     )
-    (property "Datasheet" "~" (at 188.595 40.005 0)
+    (property "Datasheet" "https://www.lcsc.com/product-detail/Tactile-Switches_E-Switch-TL3342F450QG_C2886897.html" (at 188.595 40.005 0)
       (effects (font (size 1.27 1.27)) hide)
     )
@@
       (effects (font (size 0.508 0.508)) hide)
     )
-    (property "Datasheet" "" (at 126.365 180.34 0)
+    (property "Datasheet" "https://www.lcsc.com/product-detail/Chip-Resistor-Surface-Mount_VO-SCR0402J0R_C3017451.html" (at 126.365 180.34 0)
       (effects (font (size 1.524 1.524)) hide)
     )
@@
       (effects (font (size 1.524 1.524)) (justify right))
     )
-    (property "LCSC_Part_Number" "C163812" (at 126.365 180.34 0)
+    (property "LCSC_Part_Number" "C3017451" (at 126.365 180.34 0)
       (effects (font (size 1.27 1.27)) hide)
     )
@@
       (effects (font (size 0.508 0.508)) hide)
     )
-    (property "Datasheet" "" (at 34.925 174.625 0)
+    (property "Datasheet" "https://www.lcsc.com/product-detail/Chip-Resistor-Surface-Mount_FOJAN-FRC0402J102-TS_C2906899.html" (at 34.925 174.625 0)
       (effects (font (size 1.524 1.524)) hide)
     )
@@
       (effects (font (size 1.524 1.524)) (justify right))
     )
-    (property "LCSC_Part_Number" "C100195" (at 34.925 174.625 0)
+    (property "LCSC_Part_Number" "C2906899" (at 34.925 174.625 0)
       (effects (font (size 1.27 1.27)) hide)
     )
@@
       (effects (font (size 0.508 0.508)) hide)
     )
-    (property "Datasheet" "" (at 125.73 155.575 0)
+    (property "Datasheet" "https://www.lcsc.com/product-detail/Chip-Resistor-Surface-Mount_VO-SCR0402J0R_C3017451.html" (at 125.73 155.575 0)
       (effects (font (size 1.524 1.524)) hide)
     )
@@
       (effects (font (size 1.524 1.524)) (justify right))
     )
-    (property "LCSC_Part_Number" "C163812" (at 125.73 155.575 0)
-      (effects (font (size 1.27 1.27)) hide)
-    )
+    (property "LCSC_Part_Number" "C3017451" (at 125.73 155.575 0)
+      (effects (font (size 1.27 1.27)) hide)
+    )
