File: motorgo_plink/motorgo_plink.kicad_sch (KiCad schematic)
At the start: 21 parts, among them J1 USB4520-03-0-A_REVA, J12 Conn_01x04_Pin, J4 Conn_02x20_Odd_Even, J5 Conn_01x04_Pin, J9 Conn_01x04_Pin, U1 ESP32-S3-WROOM-1, U2 USBLC6-2P6

Commit message: update to recent production files
Parts:
- D1: value LED -> LED GREEN
- D2: value LED -> LED BLUE
- D3: value LED -> LED RED
- J12, J5, J9: now not fitted
- J2, J3: value ~ -> C2886897
Connections:
- net gpio41: now also D2.2 (A)
- net gpio42: now also D1.2 (A), J4.8 (Pin_8); no longer J4.9 (Pin_9)
- net gpio43: now also J4.9 (Pin_9); no longer D2.2 (A), J4.7 (Pin_7)
- net gpio44: now also J4.7 (Pin_7); no longer D1.2 (A), J4.8 (Pin_8)
Other:
- note added: "piRX"
- note added: "piTX"
Changed lines of the file:
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@@
 	(wire
 		(pts
+			(xy 238.76 33.02) (xy 238.125 33.02)
+		)
+		(stroke
+			(width 0)
+			(type default)
+		)
+	)
+	(wire
+		(pts
 			(xy 238.125 63.5) (xy 238.76 63.5)
 		)
@@
 		)
 	)
+	(text_box "data_ready"
+		(exclude_from_sim no)
+		(at 247.65 46.99 0)
+		(size 11.43 2.54)
+		(stroke
+			(width 0)
+			(type default)
+		)
+		(fill
+			(type none)
+		)
+		(effects
+			(font
+				(size 1.27 1.27)
+			)
+			(justify left top)
+		)
+	)
+	(text_box "CLK"
+		(exclude_from_sim no)
+		(at 208.28 49.53 0)
+		(size 6.35 2.54)
+		(stroke
+			(width 0)
+			(type default)
+		)
+		(fill
+			(type none)
+		)
+		(effects
+			(font
+				(size 1.27 1.27)
+			)
+			(justify left top)
+		)
+	)
+	(text_box "CS"
+		(exclude_from_sim no)
+		(at 247.65 49.53 0)
+		(size 6.35 2.54)
+		(stroke
+			(width 0)
+			(type default)
+		)
+		(fill
+			(type none)
+		)
+		(effects
+			(font
+				(size 1.27 1.27)
+			)
+			(justify left top)
+		)
+	)
+	(text_box "COPI"
+		(exclude_from_sim no)
+		(at 208.28 44.45 0)
+		(size 6.35 2.54)
+		(stroke
+			(width 0)
+			(type default)
+		)
+		(fill
+			(type none)
+		)
+		(effects
+			(font
+				(size 1.27 1.27)
+			)
+			(justify left top)
+		)
+	)
+	(text_box "CIPO"
+		(exclude_from_sim no)
+		(at 208.28 46.99 0)
+		(size 6.35 2.54)
+		(stroke
+			(width 0)
+			(type default)
+		)
+		(fill
+			(type none)
+		)
+		(effects
+			(font
+				(size 1.27 1.27)
+			)
+			(justify left top)
+		)
+	)
 	(text "USB-C Programming connector\n"
 		(exclude_from_sim no)
@@
 		)
 	)
+	(text "piRX"
+		(exclude_from_sim no)
+		(at 250.698 33.02 0)
+		(effects
+			(font
+				(size 1.27 1.27)
+			)
+		)
+	)
+	(text "piTX"
+		(exclude_from_sim no)
+		(at 250.698 30.226 0)
+		(effects
+			(font
+				(size 1.27 1.27)
+			)
+		)
+	)
 	(text "The ADC2 Channels do not\nperform as expected with the wifi capabilities of the ESP32"
 		(exclude_from_sim no)
@@
 		)
 	)
+	(global_label "gpio42"
+		(shape input)
+		(at 25.4 137.16 180)
+		(fields_autoplaced yes)
+		(effects
+			(font
+				(size 1.27 1.27)
+			)
+			(justify right)
+		)
+		(property "Intersheetrefs" "${INTERSHEET_REFS}"
+			(at 15.944 137.16 0)
+			(effects
+				(font
+					(size 1.27 1.27)
+				)
+				(justify right)
+				(hide yes)
+			)
+		)
+	)
 	(global_label "m4_EN"
 		(shape input)
@@
 		)
 	)
-	(global_label "gpio44"
-		(shape input)
-		(at 25.4 137.16 0)
-		(fields_autoplaced yes)
-		(effects
-			(font
-				(size 1.27 1.27)
-			)
-			(justify left)
-		)
-		(property "Intersheetrefs" "${INTERSHEET_REFS}"
-			(at 34.856 137.16 0)
-			(effects
-				(font
-					(size 1.27 1.27)
-				)
-				(justify left)
-				(hide yes)
-			)
-		)
-	)
 	(global_label "usb_d+"
 		(shape input)
@@
 	(global_label "gpio42"
 		(shape input)
-		(at 238.125 33.02 0)
+		(at 225.425 30.48 180)
 		(fields_autoplaced yes)
 		(effects
@@
 				(size 1.27 1.27)
 			)
-			(justify left)
+			(justify right)
 		)
 		(property "Intersheetrefs" "${INTERSHEET_REFS}"
-			(at 247.581 33.02 0)
+			(at 215.969 30.48 0)
 			(effects
 				(font
 					(size 1.27 1.27)
 				)
-				(justify left)
+				(justify right)
 				(hide yes)
 			)
@@
 		)
 	)
+	(global_label "gpio41"
+		(shape input)
+		(at 34.29 140.97 0)
+		(fields_autoplaced yes)
+		(effects
+			(font
+				(size 1.27 1.27)
+			)
+			(justify left)
+		)
+		(property "Intersheetrefs" "${INTERSHEET_REFS}"
+			(at 43.746 140.97 0)
+			(effects
+				(font
+					(size 1.27 1.27)
+				)
+				(justify left)
+				(hide yes)
+			)
+		)
+	)
 	(global_label "gpio21"
 		(shape input)
@@
 	(global_label "gpio44"
 		(shape input)
-		(at 225.425 30.48 180)
+		(at 238.76 30.48 0)
 		(fields_autoplaced yes)
 		(effects
@@
 				(size 1.27 1.27)
 			)
-			(justify right)
+			(justify left)
 		)
 		(property "Intersheetrefs" "${INTERSHEET_REFS}"
-			(at 215.969 30.48 0)
+			(at 248.216 30.48 0)
 			(effects
 				(font
 					(size 1.27 1.27)
 				)
-				(justify right)
+				(justify left)
 				(hide yes)
 			)
@@
 	(global_label "gpio43"
 		(shape input)
-		(at 238.76 30.48 0)
+		(at 238.76 33.02 0)
 		(fields_autoplaced yes)
 		(effects
@@
 		)
 		(property "Intersheetrefs" "${INTERSHEET_REFS}"
-			(at 248.216 30.48 0)
+			(at 248.216 33.02 0)
 			(effects
 				(font
@@
 		)
 	)
-	(global_label "gpio43"
-		(shape input)
-		(at 34.29 140.97 0)
-		(fields_autoplaced yes)
-		(effects
-			(font
-				(size 1.27 1.27)
-			)
-			(justify left)
-		)
-		(property "Intersheetrefs" "${INTERSHEET_REFS}"
-			(at 43.746 140.97 0)
-			(effects
-				(font
-					(size 1.27 1.27)
-				)
-				(justify left)
-				(hide yes)
-			)
-		)
-	)
 	(global_label "gpio21"
 		(shape input)
@@
 		(in_bom yes)
 		(on_board yes)
-		(dnp no)
+		(dnp yes)
 		(property "Reference" "J5"
 			(at 171.958 70.612 0)
@@
 			)
 		)
-		(property "Value" "LED"
-			(at 46.99 168.5925 90)
+		(property "Value" "LED RED"
+			(at 46.736 168.148 90)
 			(effects
 				(font
@@
 			)
 		)
-		(property "Value" "LED"
-			(at 27.94 168.5925 90)
+		(property "Value" "LED GREEN"
+			(at 19.812 168.148 90)
 			(effects
 				(font
@@
 		(in_bom yes)
 		(on_board yes)
-		(dnp no)
+		(dnp yes)
 		(property "Reference" "J9"
 			(at 179.832 70.612 0)
@@
 			)
 		)
-		(property "Value" "LED"
-			(at 38.1 168.5925 90)
+		(property "Value" "LED BLUE"
+			(at 32.258 167.894 90)
 			(effects
 				(font
@@
 			)
 		)
-		(property "Value" "~"
+		(property "Value" "C2886897"
 			(at 167.64 40.005 0)
 			(effects
@@
 		(in_bom yes)
 		(on_board yes)
-		(dnp no)
+		(dnp yes)
 		(property "Reference" "J12"
 			(at 187.452 70.612 0)
@@
 			)
 		)
-		(property "Value" "~"
+		(property "Value" "C2886897"
 			(at 183.515 40.005 0)
 			(effects
