File: motorgo_plink/plink_connectors_hs.kicad_sch (KiCad schematic)
At the start: 14 parts, among them J12 BM05B-SRSS-TB_LF__SN_, J13 BM05B-SRSS-TB_LF__SN_, J3 I2C_STANDARDQWIIC, J5 I2C_STANDARDQWIIC

Commit message: WIP update. Parts semi-finalized
Parts:
- J3, J5: footprint aa_sparkfun_connectors:1X04_1MM_RA -> Connector_JST:JST_SH_BM04B-SRSS-TB_1x04-1MP_P1.00mm_Vertical

Commit message: WIP update. Ready for BOM editing
Parts:
- removed R28, R29: 5k1, Resistor_SMD:R_0402_1005Metric, symbol sparkfun_resistors:RESISTOR0603
- added J4: Conn_02x20_Odd_Even, Connector_PinSocket_2.54mm:PinSocket_2x20_P2.54mm_Vertical_SMD, symbol Connector_Generic:Conn_02x20_Odd_Even
Connections:
- net +3.3V: now also J4.18 (Pin_18), J4.2 (Pin_2)
- net GND: now also J4.10 (Pin_10), J4.13 (Pin_13), J4.19 (Pin_19), J4.26 (Pin_26), J4.29 (Pin_29), J4.33 (Pin_33), J4.40 (Pin_40), J4.5 (Pin_5)
- net scl: now also J4.6 (Pin_6)
- net sda: now also J4.4 (Pin_4)
- new net +5V: J4.1 (Pin_1), J4.3 (Pin_3)
- new net Reset: J4.16 (Pin_16)
- new net boot: J4.30 (Pin_30)
- new net gpio3: J4.15 (Pin_15)
- new net gpio38: J4.23 (Pin_23)
- new net gpio39: J4.22 (Pin_22)
- new net gpio4: J4.11 (Pin_11)
- new net gpio40: J4.24 (Pin_24)
- new net gpio41: J4.21 (Pin_21)
- new net gpio42: J4.20 (Pin_20)
- new net gpio43: J4.9 (Pin_9)
- new net gpio44: J4.7 (Pin_7)
- new net gpio47: J4.12 (Pin_12)
- new net gpio7: J4.14 (Pin_14)
- new net gpio8: J4.17 (Pin_17)
- new net gpio9: J4.8 (Pin_8)
- new net p26: J4.25 (Pin_25)
- new net p31: J4.32 (Pin_32)
- new net p32: J4.31 (Pin_31)
- new net p33: J4.34 (Pin_34)
- new net p35: J4.36 (Pin_36)
- new net p36: J4.35 (Pin_35)
- new net p37: J4.38 (Pin_38)
- new net p38: J4.37 (Pin_37)
- new net p40: J4.39 (Pin_39)
- no-connect marks 0 -> 2
Other:
- note added: "Bottom link to Rpi"
- note added: "Pass through pins"

Commit message: WIP - adding P/Ns to BOM (TS). will finish in afternoon.
Parts:
- J4: Field4 (none) -> replaced with female (TS) 5-31; LCSC_Part_Number (none) -> C2977589
Changed lines of the file:
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@@
       (effects (font (size 1.27 1.27)) (justify left bottom) hide)
     )
-    (property "Datasheet" "" (at 108.585 70.485 0)
+    (property "Datasheet" "https://www.lcsc.com/product-detail/Wire-To-Board-Connector_JST-BM05B-SRSS-TBT-LF-SN_C265092.html" (at 108.585 70.485 0)
       (effects (font (size 1.27 1.27)) (justify left bottom) hide)
     )
@@
       (effects (font (size 1.27 1.27)) (justify left bottom) hide)
     )
-    (property "Datasheet" "" (at 76.835 70.485 0)
+    (property "Datasheet" "https://www.lcsc.com/product-detail/Wire-To-Board-Connector_JST-BM05B-SRSS-TBT-LF-SN_C265092.html" (at 76.835 70.485 0)
       (effects (font (size 1.27 1.27)) (justify left bottom) hide)
     )
@@
       (effects (font (size 1.27 1.27)) (justify left bottom) hide)
     )
-    (property "Datasheet" "" (at 46.355 70.485 0)
+    (property "Datasheet" "https://www.lcsc.com/product-detail/Wire-To-Board-Connector_JST-BM05B-SRSS-TBT-LF-SN_C265092.html" (at 46.355 70.485 0)
       (effects (font (size 1.27 1.27)) (justify left bottom) hide)
     )
@@
       (effects (font (size 0.508 0.508)) hide)
     )
-    (property "Datasheet" "" (at 40.64 130.175 0)
+    (property "Datasheet" "https://www.lcsc.com/product-detail/Wire-To-Board-Connector_JST-SM04B-SRSS-TB-LF-SN_C160404.html" (at 40.64 130.175 0)
       (effects (font (size 1.27 1.27)) hide)
     )
@@
       (effects (font (size 0.508 0.508)) hide)
     )
-    (property "Datasheet" "" (at 67.31 130.175 0)
+    (property "Datasheet" "https://www.lcsc.com/product-detail/Wire-To-Board-Connector_JST-SM04B-SRSS-TB-LF-SN_C160404.html" (at 67.31 130.175 0)
       (effects (font (size 1.27 1.27)) hide)
     )
@@
       (effects (font (size 0.508 0.508)) hide)
     )
-    (property "Datasheet" "" (at 116.205 130.175 0)
+    (property "Datasheet" "https://www.lcsc.com/product-detail/Wire-To-Board-Connector_JST-SM04B-SRSS-TB-LF-SN_C160404.html" (at 116.205 130.175 0)
       (effects (font (size 1.27 1.27)) hide)
     )
@@
       (effects (font (size 0.508 0.508)) hide)
     )
-    (property "Datasheet" "" (at 89.535 130.175 0)
+    (property "Datasheet" "https://www.lcsc.com/product-detail/Wire-To-Board-Connector_JST-SM04B-SRSS-TB-LF-SN_C160404.html" (at 89.535 130.175 0)
       (effects (font (size 1.27 1.27)) hide)
     )
@@
       (effects (font (size 1.27 1.27)) (justify left bottom) hide)
     )
-    (property "Datasheet" "" (at 139.065 70.485 0)
+    (property "Datasheet" "https://www.lcsc.com/product-detail/Wire-To-Board-Connector_JST-BM05B-SRSS-TBT-LF-SN_C265092.html" (at 139.065 70.485 0)
       (effects (font (size 1.27 1.27)) (justify left bottom) hide)
     )
@@
       (effects (font (size 1.27 1.27)) hide)
     )
-    (property "Datasheet" "~" (at 201.295 53.34 0)
-      (effects (font (size 1.27 1.27)) hide)
-    )
+    (property "Datasheet" "https://www.lcsc.com/product-detail/Female-Headers_ZHOURI-2-54-2-20_C2977589.html" (at 201.295 53.34 0)
+      (effects (font (size 1.27 1.27)) hide)
+    )
+    (property "Field4" "replaced with female (TS) 5-31" (at 201.295 53.34 0)
+      (effects (font (size 1.27 1.27)) hide)
+    )
+    (property "LCSC_Part_Number" "C2977589" (at 201.295 53.34 0)
+      (effects (font (size 1.27 1.27)) hide)
+    )

Commit message: finished first pass on BOM. check 100uF cap and a couple others. TS
Parts:
- R26, R27, R28, R29: Field4 (none) -> (none)
Changed lines of the file:
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@@
       (effects (font (size 0.508 0.508)) hide)
     )
-    (property "Datasheet" "" (at 95.25 48.895 0)
+    (property "Datasheet" "https://www.lcsc.com/product-detail/Chip-Resistor-Surface-Mount_Viking-Tech-CR-02FL6-5K1_C409700.html" (at 95.25 48.895 0)
       (effects (font (size 1.524 1.524)) hide)
     )
-    (property "Field4" " " (at 95.885 49.53 90)
+    (property "Field4" "" (at 95.885 49.53 90)
       (effects (font (size 1.524 1.524)) (justify right))
     )
@@
       (effects (font (size 0.508 0.508)) hide)
     )
-    (property "Datasheet" "" (at 51.435 113.665 0)
+    (property "Datasheet" "https://www.lcsc.com/product-detail/Chip-Resistor-Surface-Mount_Viking-Tech-CR-02FL6-5K1_C409700.html" (at 51.435 113.665 0)
       (effects (font (size 1.524 1.524)) hide)
     )
-    (property "Field4" " " (at 48.895 110.49 90)
+    (property "Field4" "" (at 48.895 110.49 90)
       (effects (font (size 1.524 1.524)) (justify right))
     )
@@
       (effects (font (size 0.508 0.508)) hide)
     )
-    (property "Datasheet" "" (at 48.895 113.665 0)
+    (property "Datasheet" "https://www.lcsc.com/product-detail/Chip-Resistor-Surface-Mount_Viking-Tech-CR-02FL6-5K1_C409700.html" (at 48.895 113.665 0)
       (effects (font (size 1.524 1.524)) hide)
     )
-    (property "Field4" " " (at 46.355 110.49 90)
+    (property "Field4" "" (at 46.355 110.49 90)
       (effects (font (size 1.524 1.524)) (justify right))
     )
@@
       (effects (font (size 0.508 0.508)) hide)
     )
-    (property "Datasheet" "" (at 97.79 48.895 0)
+    (property "Datasheet" "https://www.lcsc.com/product-detail/Chip-Resistor-Surface-Mount_Viking-Tech-CR-02FL6-5K1_C409700.html" (at 97.79 48.895 0)
       (effects (font (size 1.524 1.524)) hide)
     )
-    (property "Field4" " " (at 95.25 45.72 90)
+    (property "Field4" "" (at 95.25 45.72 90)
       (effects (font (size 1.524 1.524)) (justify right))
     )

Commit message: replaced female 2x20 header with brick nogging. male pin headers listed in the google sheets.
Parts:
- J4: LCSC_Part_Number C2977589 -> C3975165
Changed lines of the file:
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@@
       (effects (font (size 1.27 1.27)) hide)
     )
-    (property "Datasheet" "https://www.lcsc.com/product-detail/Female-Headers_ZHOURI-2-54-2-20_C2977589.html" (at 201.295 53.34 0)
+    (property "Datasheet" "https://www.lcsc.com/product-detail/Female-Headers_HCTL-PM254-2-20-S-8-5_C3975165.html" (at 201.295 53.34 0)
       (effects (font (size 1.27 1.27)) hide)
     )
@@
       (effects (font (size 1.27 1.27)) hide)
     )
-    (property "LCSC_Part_Number" "C2977589" (at 201.295 53.34 0)
+    (property "LCSC_Part_Number" "C3975165" (at 201.295 53.34 0)
       (effects (font (size 1.27 1.27)) hide)
     )
