File: motorgo_plink/plink_connectors_hs.kicad_sch (KiCad schematic)
At the start: 13 parts, among them J12 BM05B-SRSS-TB_LF__SN_, J13 BM05B-SRSS-TB_LF__SN_, J3 I2C_STANDARDQWIIC, J4 Conn_02x20_Odd_Even, J5 I2C_STANDARDQWIIC

Commit message: updated BOM in prep for order - TS
Parts:
- J4: LCSC_Part_Number (none) -> C3975165
Changed lines of the file:
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@@
       (effects (font (size 1.27 1.27)) (justify left bottom) hide)
     )
-    (property "Datasheet" "" (at 108.585 70.485 0)
+    (property "Datasheet" "https://www.lcsc.com/product-detail/Wire-To-Board-Connector_JST-BM05B-SRSS-TBT-LF-SN_C265092.html" (at 108.585 70.485 0)
       (effects (font (size 1.27 1.27)) (justify left bottom) hide)
     )
@@
       (effects (font (size 1.27 1.27)) (justify left bottom) hide)
     )
-    (property "Datasheet" "" (at 76.835 70.485 0)
+    (property "Datasheet" "https://www.lcsc.com/product-detail/Wire-To-Board-Connector_JST-BM05B-SRSS-TBT-LF-SN_C265092.html" (at 76.835 70.485 0)
       (effects (font (size 1.27 1.27)) (justify left bottom) hide)
     )
@@
       (effects (font (size 1.27 1.27)) (justify left bottom) hide)
     )
-    (property "Datasheet" "" (at 46.355 70.485 0)
+    (property "Datasheet" "https://www.lcsc.com/product-detail/Wire-To-Board-Connector_JST-BM05B-SRSS-TBT-LF-SN_C265092.html" (at 46.355 70.485 0)
       (effects (font (size 1.27 1.27)) (justify left bottom) hide)
     )
@@
       (effects (font (size 0.508 0.508)) hide)
     )
-    (property "Datasheet" "" (at 95.25 48.895 0)
+    (property "Datasheet" "https://www.lcsc.com/product-detail/Chip-Resistor-Surface-Mount_Viking-Tech-CR-02FL6-5K1_C409700.html" (at 95.25 48.895 0)
       (effects (font (size 1.524 1.524)) hide)
     )
@@
       (effects (font (size 0.508 0.508)) hide)
     )
-    (property "Datasheet" "" (at 40.64 130.175 0)
+    (property "Datasheet" "https://www.lcsc.com/product-detail/Wire-To-Board-Connector_JST-SM04B-SRSS-TB-LF-SN_C160404.html" (at 40.64 130.175 0)
       (effects (font (size 1.27 1.27)) hide)
     )
@@
       (effects (font (size 0.508 0.508)) hide)
     )
-    (property "Datasheet" "" (at 51.435 113.665 0)
+    (property "Datasheet" "https://www.lcsc.com/product-detail/Chip-Resistor-Surface-Mount_Viking-Tech-CR-02FL6-5K1_C409700.html" (at 51.435 113.665 0)
       (effects (font (size 1.524 1.524)) hide)
     )
@@
       (effects (font (size 0.508 0.508)) hide)
     )
-    (property "Datasheet" "" (at 67.31 130.175 0)
+    (property "Datasheet" "https://www.lcsc.com/product-detail/Wire-To-Board-Connector_JST-SM04B-SRSS-TB-LF-SN_C160404.html" (at 67.31 130.175 0)
       (effects (font (size 1.27 1.27)) hide)
     )
@@
       (effects (font (size 0.508 0.508)) hide)
     )
-    (property "Datasheet" "" (at 48.895 113.665 0)
+    (property "Datasheet" "https://www.lcsc.com/product-detail/Chip-Resistor-Surface-Mount_Viking-Tech-CR-02FL6-5K1_C409700.html" (at 48.895 113.665 0)
       (effects (font (size 1.524 1.524)) hide)
     )
@@
       (effects (font (size 0.508 0.508)) hide)
     )
-    (property "Datasheet" "" (at 116.205 130.175 0)
+    (property "Datasheet" "https://www.lcsc.com/product-detail/Wire-To-Board-Connector_JST-SM04B-SRSS-TB-LF-SN_C160404.html" (at 116.205 130.175 0)
       (effects (font (size 1.27 1.27)) hide)
     )
@@
       (effects (font (size 0.508 0.508)) hide)
     )
-    (property "Datasheet" "" (at 89.535 130.175 0)
+    (property "Datasheet" "https://www.lcsc.com/product-detail/Wire-To-Board-Connector_JST-SM04B-SRSS-TB-LF-SN_C160404.html" (at 89.535 130.175 0)
       (effects (font (size 1.27 1.27)) hide)
     )
@@
       (effects (font (size 1.27 1.27)) (justify left bottom) hide)
     )
-    (property "Datasheet" "" (at 139.065 70.485 0)
+    (property "Datasheet" "https://www.lcsc.com/product-detail/Wire-To-Board-Connector_JST-BM05B-SRSS-TBT-LF-SN_C265092.html" (at 139.065 70.485 0)
       (effects (font (size 1.27 1.27)) (justify left bottom) hide)
     )
@@
       (effects (font (size 1.27 1.27)) hide)
     )
-    (property "Datasheet" "~" (at 201.295 53.34 0)
+    (property "Datasheet" "https://www.lcsc.com/product-detail/Female-Headers_HCTL-PM254-2-20-S-8-5_C3975165.html" (at 201.295 53.34 0)
+      (effects (font (size 1.27 1.27)) hide)
+    )
+    (property "LCSC_Part_Number" "C3975165" (at 201.295 53.34 0)
       (effects (font (size 1.27 1.27)) hide)
     )
@@
       (effects (font (size 0.508 0.508)) hide)
     )
-    (property "Datasheet" "" (at 97.79 48.895 0)
+    (property "Datasheet" "https://www.lcsc.com/product-detail/Chip-Resistor-Surface-Mount_Viking-Tech-CR-02FL6-5K1_C409700.html" (at 97.79 48.895 0)
       (effects (font (size 1.524 1.524)) hide)
     )
