File: motorgo_plink/H_brdige_AP30H80Q.kicad_sch (KiCad schematic)
At the start: 11 parts, among them J17 Conn_01x03_Socket, J5 Conn_01x02_Pin, U3 DRV8874PWPR

Commit message: WIP update for BOM co-work
Changed lines of the file:
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@@
     (fill (type none))
   )
-  (rectangle (start 92.075 110.49) (end 120.65 131.445)
+  (rectangle (start 92.075 109.855) (end 120.65 131.445)
     (stroke (width 0) (type default))
     (fill (type none))
@@
   )
   (text "Vref = 3v3\nR_PROP = \n3v3/ 0.455 / Imax_lim" (at 93.98 116.84 0)
-    (effects (font (size 1.27 1.27)) (justify left bottom))
+    (effects (font (size 1.27 1.27) (color 255 157 178 1)) (justify left bottom))
   )
   (text "TBD connector for motors" (at 165.1 117.475 0)
-    (effects (font (size 1.27 1.27)) (justify left bottom))
+    (effects (font (size 1.27 1.27) (color 255 178 0 1)) (justify left bottom))
   )
   (text "Imax = 1.5\n=) R_prop = 4.83K" (at 93.98 126.365 0)
-    (effects (font (size 1.27 1.27)) (justify left bottom))
+    (effects (font (size 1.27 1.27) (color 160 224 255 1)) (justify left bottom))
   )
   (text "R    Imax reaction \n20k  chop & retry\n0    pause & retry\n62k  chop & latch\nhiz  pause and latch"

Commit message: WIP update, schematic mainly complete
Changed lines of the file:
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@@
     (stroke (width 0) (type default))
   )
-  (polyline (pts (xy 134.62 118.11) (xy 156.21 118.11))
+  (polyline (pts (xy 134.62 118.11) (xy 156.845 118.11))
     (stroke (width 0) (type default))
   )
@@
     (fill (type none))
   )
-  (rectangle (start 134.62 116.205) (end 156.21 127)
+  (rectangle (start 134.62 116.205) (end 156.845 127)
     (stroke (width 0) (type default))
     (fill (type none))
@@
   (text "R    Imax reaction \n20k  chop & retry\n0    pause & retry\n62k  chop & latch\nhiz  pause and latch"
     (at 135.255 127 0)
-    (effects (font (face "Cascadia Mono") (size 1.27 1.27)) (justify left bottom))
+    (effects (font (face "Monospac821 BT") (size 1.27 1.27)) (justify left bottom))
   )
   (text "C_bulk\n1000uF to 4000uF" (at 187.325 106.045 0)

Commit message: WIP update. Parts semi-finalized
Parts:
- C10: renamed from C6; footprint (none) -> Capacitor_SMD:C_Elec_10x10.2
- C7: renamed from C19; footprint (none) -> Capacitor_SMD:C_0402_1005Metric
- C8: renamed from C23; footprint (none) -> Capacitor_SMD:C_0402_1005Metric
- C9: renamed from C2; footprint (none) -> Capacitor_SMD:C_0402_1005Metric
- J7: renamed from J17; footprint (none) -> Connector_PinHeader_2.54mm:PinHeader_1x03_P2.54mm_Vertical
- J8: renamed from J5; footprint (none) -> Connector_PinHeader_2.54mm:PinHeader_1x02_P2.54mm_Vertical
- R12: renamed from R2; footprint (none) -> Resistor_SMD:R_0402_1005Metric
- R13: renamed from R29; footprint (none) -> Resistor_SMD:R_0402_1005Metric
- Rmode2: renamed from Rmode; footprint (none) -> Resistor_SMD:R_0402_1005Metric
- Rp2: renamed from Rp1; footprint (none) -> Resistor_SMD:R_0402_1005Metric
- U4: renamed from U3; footprint kicad_lceda:HTSSOP-16_L5.0-W4.4-P0.65-LS6.4-BL-EP -> LCSC_parts:HTSSOP-16_L5.0-W4.4-P0.65-LS6.4-BL-EP

Commit message: WIP update. Layout begin
Parts:
- removed C10: 1000uF, Capacitor_SMD:C_Elec_10x10.2, symbol Device:C_Polarized_US
- removed J7: Conn_01x03_Socket, Connector_PinHeader_2.54mm:PinHeader_1x03_P2.54mm_Vertical, symbol Connector:Conn_01x03_Socket
- added C10: 100uF, Capacitor_SMD:C_1210_3225Metric, symbol Device:C_Small
- added TP1, TP5, TP9: TestPoint, TestPoint:TestPoint_Pad_1.0x1.0mm, symbol Connector:TestPoint
Connections:
- net +3V3: now also TP9.1
- net +BATT: now also C10.1
- net GND: now also C10.2
- net at U4.3 (nSLEEP): now also TP1.1
- net at R12.2, U4.4 (nFAULT): now also TP5.1
Other:
- note removed: "C_bulk 1000uF to 4000uF"

Commit message: WIP update. Ready for BOM editing
Connections:
- net +3V3 renamed +3.3V
Changed lines of the file:
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@@
-    )
-  )
-  (symbol (lib_id "power:+3V3") (at 108.585 102.87 0) (unit 1)
-    (in_bom yes) (on_board yes) (dnp no) (fields_autoplaced)
-    (property "Reference" "#PWR038" (at 108.585 106.68 0)
-      (effects (font (size 1.27 1.27)) hide)
-    )
-    (property "Value" "+3V3" (at 108.585 99.695 0)
-      (effects (font (size 1.27 1.27)))
-    )
-    (property "Footprint" "" (at 108.585 102.87 0)
-      (effects (font (size 1.27 1.27)) hide)
-    )
-    (property "Datasheet" "" (at 108.585 102.87 0)
-      (effects (font (size 1.27 1.27)) hide)
-    )
-    (pin "1")
-    (instances
-      (project "motorgo_plink"
-        (path "/e63e39d7-6ac0-4ffd-8aa3-1841a4541b55/47ec5f88-3723-4b64-bf75-8726c250fd67"
-          (reference "#PWR038") (unit 1)
-        )
-        (path "/e63e39d7-6ac0-4ffd-8aa3-1841a4541b55/809f09f1-433b-4e98-96ef-90e5b5350895"
-          (reference "#PWR028") (unit 1)
-        )
-        (path "/e63e39d7-6ac0-4ffd-8aa3-1841a4541b55/1c707bfd-41ae-4cae-875a-703c10e57ff5"
-          (reference "#PWR048") (unit 1)
-        )
-        (path "/e63e39d7-6ac0-4ffd-8aa3-1841a4541b55/4afe8fbd-60dc-4560-bdae-30691fd6b471"
-          (reference "#PWR096") (unit 1)
-        )
-      )
     )
   )
@@
         )
       )
+    )
+  )
+  (symbol (lib_id "power:+3.3V") (at 108.585 102.87 0) (unit 1)
+    (in_bom yes) (on_board yes) (dnp no)
+    (property "Reference" "#PWR075" (at 108.585 106.68 0)
+      (effects (font (size 1.27 1.27)) hide)
+    )
+    (property "Value" "+3.3V" (at 104.775 102.87 0)
+      (effects (font (size 1.27 1.27)))
+    )
+    (property "Footprint" "" (at 108.585 102.87 0)
+      (effects (font (size 1.27 1.27)) hide)
+    )
+    (property "Datasheet" "" (at 108.585 102.87 0)
+      (effects (font (size 1.27 1.27)) hide)
+    )
+    (pin "1")
+    (instances
+      (project "motorgo_plink"
+        (path "/e63e39d7-6ac0-4ffd-8aa3-1841a4541b55/c5a81061-28ff-4599-a380-43adb8d460db"
+          (reference "#PWR075") (unit 1)
+        )
+        (path "/e63e39d7-6ac0-4ffd-8aa3-1841a4541b55/809f09f1-433b-4e98-96ef-90e5b5350895"
+          (reference "#PWR064") (unit 1)
+        )
+        (path "/e63e39d7-6ac0-4ffd-8aa3-1841a4541b55/47ec5f88-3723-4b64-bf75-8726c250fd67"
+          (reference "#PWR0119") (unit 1)
+        )
+        (path "/e63e39d7-6ac0-4ffd-8aa3-1841a4541b55/1c707bfd-41ae-4cae-875a-703c10e57ff5"
+          (reference "#PWR0120") (unit 1)
+        )
+        (path "/e63e39d7-6ac0-4ffd-8aa3-1841a4541b55/4afe8fbd-60dc-4560-bdae-30691fd6b471"
+          (reference "#PWR0121") (unit 1)
+        )
+      )

Commit message: WIP update. change USBC port
Parts:
- Rp2: value 4.83k -> 4.87k
Other:
- note added: "Imax = 1.489 =) R_prop = 4.87K"
- note removed: "Imax = 1.5 =) R_prop = 4.83K"
Changed lines of the file:
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@@
     (effects (font (size 1.27 1.27) (color 255 178 0 1)) (justify left bottom))
   )
-  (text "Imax = 1.5\n=) R_prop = 4.83K" (at 93.98 126.365 0)
+  (text "Imax = 1.489\n=) R_prop = 4.87K" (at 93.98 126.365 0)
     (effects (font (size 1.27 1.27) (color 160 224 255 1)) (justify left bottom))
   )
@@
       (effects (font (size 1.27 1.27)) (justify left))
     )
-    (property "Value" "4.83k" (at 112.395 121.92 0)
+    (property "Value" "4.87k" (at 112.395 121.92 0)
       (effects (font (size 1.27 1.27)) (justify left))
     )

Commit message: WIP (TS) - updating BOM with values from other branch.
Parts:
- C10: LCSC_Part_Number (none) -> C6120014
- C7, C8: LCSC_Part_Number (none) -> C3012377
- C9: LCSC_Part_Number (none) -> C380305
Changed lines of the file:
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@@
       (effects (font (size 1.27 1.27)) hide)
     )
-    (property "Datasheet" "~" (at 163.83 102.235 0)
+    (property "Datasheet" "https://www.lcsc.com/product-detail/Multilayer-Ceramic-Capacitors-MLCC-SMD-SMT_HRE-CSA0402X7R104K500GT_C3012377.html" (at 163.83 102.235 0)
+      (effects (font (size 1.27 1.27)) hide)
+    )
+    (property "LCSC_Part_Number" "C3012377" (at 163.83 102.235 0)
       (effects (font (size 1.27 1.27)) hide)
     )
@@
       (effects (font (size 1.27 1.27)) hide)
     )
-    (property "Datasheet" "~" (at 177.165 104.775 0)
+    (property "Datasheet" "https://www.lcsc.com/product-detail/Multilayer-Ceramic-Capacitors-MLCC-SMD-SMT_HRE-CGA1210X5R107M160RT_C6120014.html" (at 177.165 104.775 0)
+      (effects (font (size 1.27 1.27)) hide)
+    )
+    (property "LCSC_Part_Number" "C6120014" (at 177.165 104.775 0)
       (effects (font (size 1.27 1.27)) hide)
     )
@@
       (effects (font (size 1.27 1.27)) hide)
     )
-    (property "Datasheet" "~" (at 163.83 97.155 0)
+    (property "Datasheet" "https://www.lcsc.com/product-detail/Multilayer-Ceramic-Capacitors-MLCC-SMD-SMT_HRE-CSA0402X7R104K500GT_C3012377.html" (at 163.83 97.155 0)
+      (effects (font (size 1.27 1.27)) hide)
+    )
+    (property "LCSC_Part_Number" "C3012377" (at 163.83 97.155 0)
       (effects (font (size 1.27 1.27)) hide)
     )
@@
       (effects (font (size 1.27 1.27)) hide)
     )
-    (property "Datasheet" "~" (at 170.815 89.535 0)
-      (effects (font (size 1.27 1.27)) hide)
-    )
+    (property "Datasheet" "https://www.lcsc.com/product-detail/Multilayer-Ceramic-Capacitors-MLCC-SMD-SMT_CCTC-TCC0402X7R223K500AT_C380305.html" (at 170.815 89.535 0)
+      (effects (font (size 1.27 1.27)) hide)
+    )
+    (property "LCSC_Part_Number" "C380305" (at 170.815 89.535 0)
+      (effects (font (size 1.27 1.27)) hide)
+    )

Commit message: updated BOM in prep for order - TS
Parts:
- J8: LCSC_Part_Number (none) -> C7430358
- R12, R13: LCSC_Part_Number (none) -> C2906885
- Rmode2: LCSC_Part_Number (none) -> C3017501
- Rp2: LCSC_Part_Number (none) -> C3015971
- U4: LCSC_Part_Number (none) -> C1855818
Changed lines of the file:
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@@
       (effects (font (size 1.27 1.27)) hide)
     )
-    (property "Datasheet" "https://www.lcsc.com/datasheet/lcsc_datasheet_2302221400_Texas-Instruments-DRV8874PWPR_C1855818.pdf" (at 141.605 87.503 0)
+    (property "Datasheet" "https://www.lcsc.com/product-detail/Motor-Driver-ICs_Texas-Instruments-DRV8874PWPR_C1855818.html" (at 141.605 87.503 0)
       (effects (font (size 1.27 1.27)) hide)
     )
@@
     )
     (property "uuid" "std:7384bdd1e05a4b1a8e1bd8e8948bd536" (at 141.605 92.583 0)
+      (effects (font (size 1.27 1.27)) hide)
+    )
+    (property "LCSC_Part_Number" "C1855818" (at 141.605 92.71 0)
       (effects (font (size 1.27 1.27)) hide)
     )
@@
       (effects (font (size 1.27 1.27)) hide)
     )
-    (property "Datasheet" "~" (at 166.37 76.835 0)
+    (property "Datasheet" "https://www.lcsc.com/product-detail/Chip-Resistor-Surface-Mount_FOJAN-FRC0402J103-TS_C2906885.html" (at 166.37 76.835 0)
+      (effects (font (size 1.27 1.27)) hide)
+    )
+    (property "LCSC_Part_Number" "C2906885" (at 166.37 76.835 0)
       (effects (font (size 1.27 1.27)) hide)
     )
@@
       (effects (font (size 1.27 1.27)) hide)
     )
-    (property "Datasheet" "~" (at 119.38 120.015 0)
+    (property "Datasheet" "https://www.lcsc.com/product-detail/Chip-Resistor-Surface-Mount_VO-SCR0402F4K87_C3015971.html" (at 119.38 120.015 0)
+      (effects (font (size 1.27 1.27)) hide)
+    )
+    (property "LCSC_Part_Number" "C3015971" (at 119.38 120.015 0)
       (effects (font (size 1.27 1.27)) hide)
     )
@@
       (effects (font (size 1.27 1.27)) hide)
     )
-    (property "Datasheet" "~" (at 111.76 83.82 0)
+    (property "Datasheet" "https://www.lcsc.com/product-detail/Chip-Resistor-Surface-Mount_FOJAN-FRC0402J103-TS_C2906885.html" (at 111.76 83.82 0)
+      (effects (font (size 1.27 1.27)) hide)
+    )
+    (property "LCSC_Part_Number" "C2906885" (at 111.76 83.82 0)
       (effects (font (size 1.27 1.27)) hide)
     )
@@
       (effects (font (size 1.27 1.27)) hide)
     )
-    (property "Datasheet" "~" (at 188.595 128.905 0)
+    (property "Datasheet" "https://www.lcsc.com/product-detail/Pin-Headers_CONNFLY-Elec-DS1021-1x2SF11-B_C7430358.html" (at 188.595 128.905 0)
+      (effects (font (size 1.27 1.27)) hide)
+    )
+    (property "LCSC_Part_Number" "C7430358" (at 188.595 128.905 0)
       (effects (font (size 1.27 1.27)) hide)
     )
@@
       (effects (font (size 1.27 1.27)) hide)
     )
-    (property "Datasheet" "~" (at 123.19 120.015 0)
-      (effects (font (size 1.27 1.27)) hide)
-    )
+    (property "Datasheet" "https://www.lcsc.com/product-detail/Chip-Resistor-Surface-Mount_VO-SCR0402J20K_C3017501.html" (at 123.19 120.015 0)
+      (effects (font (size 1.27 1.27)) hide)
+    )
+    (property "LCSC_Part_Number" "C3017501" (at 123.19 120.015 0)
+      (effects (font (size 1.27 1.27)) hide)
+    )
