File: motorgo_plink/H_brdige_AP30H80Q.kicad_sch (KiCad schematic)
At the start: 13 parts, among them J8 Conn_01x02_Pin, U4 DRV8874PWPR

Commit message: wip schematic edits to account for buck reg design
Parts:
- removed C10: 100uF, Capacitor_SMD:C_1210_3225Metric, symbol Device:C_Small
- removed C7, C8: 0.1uF, Capacitor_SMD:C_0402_1005Metric, symbol Device:C_Small
- removed C9: .022uF, Capacitor_SMD:C_0402_1005Metric, symbol Device:C_Small
- removed J8: Conn_01x02_Pin, Connector_PinHeader_2.54mm:PinHeader_1x02_P2.54mm_Vertical, symbol Connector:Conn_01x02_Pin
- removed R12, R13: 10k, Resistor_SMD:R_0402_1005Metric, symbol Device:R
- removed Rmode2: 20k, Resistor_SMD:R_0402_1005Metric, symbol Device:R
- removed Rp2: 4.87k, Resistor_SMD:R_0402_1005Metric, symbol Device:R
- removed TP1, TP5, TP9: TestPoint, TestPoint:TestPoint_Pad_1.0x1.0mm, symbol Connector:TestPoint
- removed U4: DRV8874PWPR, LCSC_parts:HTSSOP-16_L5.0-W4.4-P0.65-LS6.4-BL-EP, symbol LCSC_imports:DRV8874PWPR
Other:
- note removed: "Imax = 1.489 =) R_prop = 4.87K"
- note removed: "R Imax reaction 20k chop & retry 0 pause & retry 62k chop & latch hiz pause and latch"
- note removed: "TBD connector for motors"
- note removed: "Vref = 3v3 R_PROP = 3v3/ 0.455 / Imax_lim"
